File: examples/fpga-audio/reviewed/fpga-audio.kicad_pcb (KiCad board)
At the start: 2 copper layers, 94 x 84 mm, 26 parts, among them J1 3V3 IN, J2 AUDIO OUT, J3 SPI PROG, U1 iCE40UP5K, U2 PCM5102A, U3 AP2112K-1.2, U4 W25Q32JV, X1 12MHz

Commit message: Finish the fifth example, and stamp the model that wrote them
All five reviewed boards now pass KiCad's own checks: no DRC errors, nothing
unconnected, no schematic-parity findings, on 9.0.9 and 10.0.4. What is left
across the whole set is four silkscreen warnings and one library-footprint
hash, all of which come from the KiCad footprints themselves.

Getting the iCE40 board there found five things, each of which was silently
producing a board that was not the board the schematic described:

* **Two nets touching on the sheet is not something an endpoint check can
  see.** A wire that ends *on* another wire joins them, and on a sheet where
  every pin drags a stub behind it that is the common case. `schematic_shorts`
  looks for it now, and found three on this design - one of which had merged
  the 1.2 V and 3.3 V rails. The only visible sign had been KiCad's parity
  check disagreeing about a net name.
* **A symbol drawn in four units has to be placed four times.** Emitting all
  forty-eight pins under `(unit 1)` leaves three quarters of them in units
  that were never placed, which is twenty-five parity findings and a sheet
  nobody can read. The iCE40's banks and its supplies are four boxes now.
* **A pin the design does not use still has a net.** KiCad names it
  `unconnected-(U1A-IOT_37a-Pad23)`; a board that leaves the pad bare disagrees
  about every one of them.
* **A QFN counts anticlockwise**, so its east and north rows run bottom-to-top
  and right-to-left, and handing them to the fan-out in number order made
  every escape on those sides cross every other one.
* **Two rectangles that meet at a corner are further apart than growing both
  and asking whether they intersect makes them look** - which is every pair of
  pads on the corner of a QFN.

And two smaller ones: the router now keeps its vias away from every drilled
hole rather than only from its own, and the degraded variant is degraded from
the *routed* design rather than re-routed, which is both th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
Parts:
- moved C9 44.9 mm to (136.0, 74.0)
- moved X1 44.9 mm to (130.0, 74.0)
- moved C1 4.00 mm to (118.0, 76.0)
Connections:
- U1 pad 10: (no net) -> unconnected-(U1B-IOB_18a-Pad10)
- U1 pad 11: (no net) -> unconnected-(U1B-IOB_20a-Pad11)
- U1 pad 12: (no net) -> unconnected-(U1B-IOB_22a-Pad12)
- U1 pad 13: (no net) -> unconnected-(U1B-IOB_24a-Pad13)
- U1 pad 18: (no net) -> unconnected-(U1B-IOB_31b-Pad18)
- U1 pad 19: (no net) -> unconnected-(U1B-IOB_29b-Pad19)
- U1 pad 2: (no net) -> unconnected-(U1C-IOB_6a-Pad2)
- U1 pad 20: /CLK12 -> unconnected-(U1B-IOB_25b_G3-Pad20)
- U1 pad 21: (no net) -> unconnected-(U1B-IOB_23b-Pad21)
- U1 pad 23: (no net) -> unconnected-(U1A-IOT_37a-Pad23)
- U1 pad 25: (no net) -> unconnected-(U1A-IOT_36b-Pad25)
- U1 pad 26: (no net) -> unconnected-(U1A-IOT_39a-Pad26)
- U1 pad 27: (no net) -> unconnected-(U1A-IOT_38b-Pad27)
- U1 pad 28: (no net) -> unconnected-(U1A-IOT_41a-Pad28)
- U1 pad 3: (no net) -> unconnected-(U1C-IOB_9b-Pad3)
- U1 pad 31: (no net) -> unconnected-(U1A-IOT_42b-Pad31)
- U1 pad 37: (no net) -> /CLK12
- U1 pad 38: (no net) -> unconnected-(U1A-IOT_50b-Pad38)
- U1 pad 39: (no net) -> unconnected-(U1A-RGB0-Pad39)
- U1 pad 4: (no net) -> unconnected-(U1C-IOB_8a-Pad4)
- U1 pad 40: (no net) -> unconnected-(U1A-RGB1-Pad40)
- U1 pad 41: (no net) -> unconnected-(U1A-RGB2-Pad41)
- U1 pad 42: (no net) -> unconnected-(U1A-IOT_51a-Pad42)
- U1 pad 43: (no net) -> unconnected-(U1A-IOT_49a-Pad43)
- U1 pad 44: (no net) -> unconnected-(U1C-IOB_3b_G6-Pad44)
- U1 pad 45: (no net) -> unconnected-(U1C-IOB_5b-Pad45)
- U1 pad 46: (no net) -> unconnected-(U1C-IOB_0a-Pad46)
- U1 pad 47: (no net) -> unconnected-(U1C-IOB_2a-Pad47)
- U1 pad 48: (no net) -> unconnected-(U1C-IOB_4a-Pad48)
- U1 pad 6: (no net) -> unconnected-(U1B-IOB_13b-Pad6)
- U1 pad 9: (no net) -> unconnected-(U1B-IOB_16a-Pad9)
- U3 pad 4: (no net) -> unconnected-(U3-NC-Pad4)
Routing:
- net +3V3: track 482.6 -> 536.9 mm, vias 8 -> 4
- net /I2S_LRCK: track 26.3 -> 49.1 mm, vias 0 -> 4
- net /SPI_SS: track 90.6 -> 73.4 mm, vias 2 -> 4
- net /SPI_SCK: track 78.2 -> 69.1 mm, vias 0 -> 2
- net /CLK12: track 38.9 -> 30.2 mm
- net /+1V2: track 136.1 -> 129.6 mm
- net /CRESET: track 104.5 -> 110.6 mm, vias 3 -> 4
- net GND: track 135.6 -> 140.8 mm, vias 34 -> 36
- net /SPI_SO: track 78.5 -> 82.2 mm, vias 4 -> 2
- net /LDOO: track 16.7 -> 20.1 mm
- net /I2S_DIN: track 27.1 -> 28.9 mm, vias 0 -> 2
- net /OUTR: track 14.5 -> 15.5 mm
- net /I2S_SCK: track 27.4 -> 28.1 mm
- net /OUTL: track 17.1 -> 17.6 mm
- net /SPI_SI: track 68.7 -> 68.4 mm, vias 4 -> 2
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
Commit message: Read the five as an engineer would, and make the toolkit act on it
examples/REVIEW.md is the pass: the five designs read for circuit theory,
layout physics and readability, every finding dispatched to one of four
places - a rule, a fix, a reasoned waiver, or named as open. The headline
result: every reviewed/ project now PASSES its own gate, every as-generated/
still fails it, and every waiver is an engineering argument a reviewer can
disagree with.

Four new rules, each calibrated against KiCad's 18 human-drawn demo projects:

* readability.label_only - the sheet connects by name, not by wire; the
  single most recognisable mark of a generated schematic. 0 findings on the
  human corpus, 71-100% on ours.
* analog.no_dc_path - a net of only capacitors and connectors has nothing
  setting its DC level. Found a real fault: the op-amp filter's AC-coupled
  output floated. 0 findings on the corpus.
* route.detour - routed copper against the MST of the net's pads; the scenic
  tour an autorouter takes. 8 human boards fired at 2.5x, 0 at the shipped 4x.
* route.return_path - signal running over cuts in the other layer's ground
  fill, computed from the difference between a zone's outline and its fill,
  which the parser now keeps. Fires on 4 real demo boards, because real
  two-layer boards genuinely have the disease.

Three rules re-judged on evidence instead of names:

* analog.missing_decoupling reads pin electrical types: only power_in pins
  ask for a capacitor, and a net an output pin drives is never asked - a cap
  on an op-amp output is somebody's control loop. Retires the VBUS/VREF
  false positives without a single waiver.
* track.thin_power measures the longest contiguous narrow run against a
  power_neck_mm allowance. Pad entries and fine-pitch escapes pass; thin
  trunks still fail. 9 demo boards fired before, 0 after - all nine were necks.
* net.single_pin honours no-connect flags: a flagged pin is a decision.

And the designs themselves got the fixes the pa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
Parts:
- added C17: 10u, Capacitor_SMD:C_0603_1608Metric, F.Cu at (159.0, 103.0)
- added R3: 100R, Resistor_SMD:R_0603_1608Metric, F.Cu at (163.0, 110.0)
- added R4: 10k, Resistor_SMD:R_0603_1608Metric, F.Cu at (156.0, 134.0)
- C12: value 1u -> 2u2
- moved C5 12.1 mm to (156.0, 103.0), turned to 90 degrees
- moved C14 5.00 mm to (184.0, 105.5)
- moved C13 4.00 mm to (184.0, 101.0), turned to 90 degrees
Connections:
- C13 pad 2: GND -> /CAPM
- C14 pad 1: /CAPM -> /VNEG
- C14 pad 2: /VNEG -> GND
- C5 pad 1: /+1V2 -> /VCCPLL
- U1 pad 29: /+1V2 -> /VCCPLL
Routing:
- net /VCCPLL: track 0.00 -> 44.8 mm, vias 0 -> 4
- net GND: track 140.8 -> 168.7 mm, vias 36 -> 37
- net /+1V2: track 129.6 -> 104.2 mm, vias 10 -> 8
- net +3V3: track 536.9 -> 561.6 mm
- net /SPI_SS: track 73.4 -> 93.9 mm
- net /VNEG: track 9.69 -> 16.7 mm
- net /CRESET: track 110.6 -> 104.7 mm, vias 4 -> 3
- net /I2S_LRCK: track 49.1 -> 45.0 mm, vias 4 -> 2
- net /SPI_SI: track 68.4 -> 70.5 mm
- net /I2S_SCK: track 28.1 -> 30.0 mm, vias 0 -> 2
- net /OUTL: track 17.6 -> 16.3 mm, vias 1 -> 0
- net /CAPP: track 9.25 -> 10.3 mm
- net /SPI_SCK: track 69.1 -> 70.0 mm
- net /OUTR: track 15.5 -> 14.7 mm, vias 0 -> 1
- net /SPI_SO: track 82.2 -> 82.9 mm
