File: examples/fpga-audio/reviewed/fpga-audio.kicad_pcb (KiCad board)
At the start: 2 copper layers, 100 x 84 mm, 29 parts, among them J1 3V3 IN, J2 AUDIO OUT, J3 SPI PROG, U1 iCE40UP5K, U2 PCM5102A, U3 AP2112K-1.2, U4 W25Q32JV, X1 12MHz

Commit message: Measure the copper that goes out and comes back, and the text drawn on text
The reviewer sent screenshots with circles on them. Two kinds: strings
printed through each other on the schematics, and copper that leaves a
pad, travels three sides of a rectangle and arrives four millimetres
away. Neither had a rule that could see it - `text_over_wire` measured
text against nets and nothing measured text against text, and
`route.detour` weighs a whole net, which averages one bad connection
away under any ratio worth setting.

New rule `route.wander`: one continuous run of copper - pad or junction
at each end - against the shortest way between those two ends that
clears the packages in between. The baseline walks the perimeter of
whatever the straight line crosses, so an opamp's feedback wrap is
measured against going round the package rather than through it. On
KiCad's 18 demo boards it fires once at the shipped 2.0x.

`readability.text_over_text` and `_over_wire` are regraded info: they
fire on 14 and 10 of those 18 human sheets. That is the estimate
talking, not the drawing. `ai-generated` still promotes both to errors,
so every generated design has to have none - and the five examples do.

What the two rules then made us fix:

* a net label's anchor cannot move, but its reading direction can. Each
  name is now offered the four quarters of its anchor and takes the
  first that prints over nothing. Power symbol names and PWR_FLAG names
  get the same treatment - four grounds on one row printed GNGNGNGND.
  Schematic text overlaps: buck 1, motor 2, carrier 1, fpga 7, all to 0.
* a plane crossing was priced at forty times front copper per
  millimetre, which is a prohibition, not a price: one millimetre of
  crossing bought a forty millimetre tour and the boards had grown
  them. Thirty is where neither `route.wander` nor `route.return_path`
  fires. Buck, motor and carrier now have no wander findings.
* `write_variant` resolves the routes a second time, so the
  straight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
Routing:
- net /CRESET: track 162.7 -> 141.8 mm
- net +3V3: track 629.1 -> 615.0 mm
- net GND: track 134.5 -> 134.2 mm, vias 173 -> 170
Changed lines of the file:
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@@
 	(segment (start 136.1 133.905) (end 135.005 135.0) (width 0.2) (layer "F.Cu") (net 1))
 	(segment (start 135.005 135.0) (end 133.5 135.0) (width 0.2) (layer "F.Cu") (net 1))
-	(segment (start 142.475 130.095) (end 143.9 130.095) (width 0.2) (layer "F.Cu") (net 3))
-	(segment (start 143.9 130.095) (end 144.995 129.0) (width 0.2) (layer "F.Cu") (net 3))
-	(segment (start 144.995 129.0) (end 146.146 129.0) (width 0.2) (layer "F.Cu") (net 3))
-	(segment (start 146.146 129.0) (end 146.146 129.146) (width 0.2) (layer "F.Cu") (net 3))
-	(segment (start 146.146 129.146) (end 146.25 129.25) (width 0.2) (layer "F.Cu") (net 3))
-	(segment (start 146.25 129.25) (end 145.75 129.25) (width 0.2) (layer "F.Cu") (net 3))
-	(segment (start 145.75 129.25) (end 145.25 128.75) (width 0.2) (layer "F.Cu") (net 3))
-	(segment (start 145.25 128.75) (end 145.25 128.25) (width 0.2) (layer "F.Cu") (net 3))
-	(segment (start 145.25 128.25) (end 145.225 128.225) (width 0.2) (layer "F.Cu") (net 3))
-	(segment (start 145.225 128.225) (end 145.225 128.0) (width 0.2) (layer "F.Cu") (net 3))
-	(segment (start 142.475 131.365) (end 143.9 131.365) (width 0.2) (layer "F.Cu") (net 3))
-	(segment (start 143.9 131.365) (end 144.65 131.365) (width 0.2) (layer "F.Cu") (net 3))
-	(segment (start 144.65 131.365) (end 145.015 131.0) (width 0.2) (layer "F.Cu") (net 3))
-	(segment (start 145.015 131.0) (end 146.5 131.0) (width 0.2) (layer "F.Cu") (net 3))
-	(segment (start 146.5 131.0) (end 147.125 130.375) (width 0.2) (layer "F.Cu") (net 3))
-	(segment (start 147.125 130.375) (end 147.125 130.009) (width 0.2) (layer "F.Cu") (net 3))
-	(segment (start 147.125 130.009) (end 146.866 129.75) (width 0.2) (layer "F.Cu") (net 3))
-	(segment (start 146.866 129.75) (end 142.75 129.75) (width 0.2) (layer "F.Cu") (net 3))
-	(segment (start 142.75 129.75) (end 139.5 133.0) (width 0.2) (layer "F.Cu") (net 3))
-	(segment (start 139.5 133.0) (end 133.5 133.0) (width 0.2) (layer "F.Cu") (net 3))
+	(segment (start 142.475 130.095) (end 143.13 130.095) (width 0.2) (layer "F.Cu") (net 3))
+	(segment (start 143.13 130.095) (end 145.225 128.0) (width 0.2) (layer "F.Cu") (net 3))
+	(segment (start 142.475 131.365) (end 133.5 133.0) (width 0.2) (layer "F.Cu") (net 3))
 	(segment (start 142.475 132.635) (end 143.9 132.635) (width 0.2) (layer "F.Cu") (net 16))
 	(segment (start 143.9 132.635) (end 144.65 132.635) (width 0.2) (layer "F.Cu") (net 16))
@@
 	(segment (start 118.0 97.0) (end 118.0 86.75) (width 0.2) (layer "F.Cu") (net 8))
 	(segment (start 118.0 86.75) (end 120.0 86.75) (width 0.2) (layer "B.Cu") (net 8))
-	(segment (start 120.0 86.75) (end 125.0 86.75) (width 0.2) (layer "F.Cu") (net 8))
-	(segment (start 125.0 86.75) (end 129.25 82.5) (width 0.2) (layer "F.Cu") (net 8))
-	(segment (start 129.25 82.5) (end 129.25 82.25) (width 0.2) (layer "F.Cu") (net 8))
-	(segment (start 129.25 82.25) (end 129.25 82.075) (width 0.2) (layer "F.Cu") (net 8))
-	(segment (start 129.25 82.075) (end 129.325 82.0) (width 0.2) (layer "F.Cu") (net 8))
-	(segment (start 129.325 82.0) (end 129.325 82.175) (width 0.2) (layer "F.Cu") (net 8))
-	(segment (start 129.325 82.175) (end 129.25 82.25) (width 0.2) (layer "F.Cu") (net 8))
-	(segment (start 129.25 82.25) (end 129.25 82.5) (width 0.2) (layer "F.Cu") (net 8))
-	(segment (start 129.25 82.5) (end 126.5 85.25) (width 0.2) (layer "F.Cu") (net 8))
-	(segment (start 126.5 85.25) (end 120.0 85.25) (width 0.2) (layer "F.Cu") (net 8))
+	(segment (start 120.0 86.75) (end 120.0 85.25) (width 0.2) (layer "F.Cu") (net 8))
 	(segment (start 120.0 85.25) (end 118.0 85.25) (width 0.2) (layer "B.Cu") (net 8))
 	(segment (start 118.0 85.25) (end 118.0 128.0) (width 0.2) (layer "F.Cu") (net 8))
@@
 	(segment (start 133.25 135.25) (end 132.5 136.0) (width 0.4) (layer "B.Cu") (net 1))
 	(segment (start 132.5 136.0) (end 130.0 136.0) (width 0.4) (layer "B.Cu") (net 1))
-	(segment (start 164.0 103.5) (end 163.625 103.125) (width 0.4) (layer "B.Cu") (net 1))
-	(segment (start 163.625 103.125) (end 162.875 103.125) (width 0.4) (layer "B.Cu") (net 1))
-	(segment (start 162.875 103.125) (end 162.5 103.5) (width 0.4) (layer "B.Cu") (net 1))
+	(segment (start 164.0 103.5) (end 162.5 103.5) (width 0.4) (layer "B.Cu") (net 1))
 	(segment (start 164.0 95.5) (end 162.5 95.5) (width 0.4) (layer "F.Cu") (net 1))
 	(segment (start 164.0 100.5) (end 162.5 100.5) (width 0.4) (layer "F.Cu") (net 1))
@@
 	(via (at 185.5 76.5) (size 0.8) (drill 0.4) (layers "F.Cu" "B.Cu") (net 1))
 	(via (at 191.5 76.5) (size 0.8) (drill 0.4) (layers "F.Cu" "B.Cu") (net 1))
-	(via (at 119.5 82.5) (size 0.8) (drill 0.4) (layers "F.Cu" "B.Cu") (net 1))
 	(via (at 125.5 82.5) (size 0.8) (drill 0.4) (layers "F.Cu" "B.Cu") (net 1))
 	(via (at 131.5 82.5) (size 0.8) (drill 0.4) (layers "F.Cu" "B.Cu") (net 1))
@@
 	(via (at 125.5 118.5) (size 0.8) (drill 0.4) (layers "F.Cu" "B.Cu") (net 1))
 	(via (at 143.5 118.5) (size 0.8) (drill 0.4) (layers "F.Cu" "B.Cu") (net 1))
-	(via (at 149.5 118.5) (size 0.8) (drill 0.4) (layers "F.Cu" "B.Cu") (net 1))
 	(via (at 155.5 118.5) (size 0.8) (drill 0.4) (layers "F.Cu" "B.Cu") (net 1))
 	(via (at 161.5 118.5) (size 0.8) (drill 0.4) (layers "F.Cu" "B.Cu") (net 1))
@@
 	(via (at 113.5 124.5) (size 0.8) (drill 0.4) (layers "F.Cu" "B.Cu") (net 1))
 	(via (at 119.5 124.5) (size 0.8) (drill 0.4) (layers "F.Cu" "B.Cu") (net 1))
-	(via (at 125.5 124.5) (size 0.8) (drill 0.4) (layers "F.Cu" "B.Cu") (net 1))
 	(via (at 137.5 124.5) (size 0.8) (drill 0.4) (layers "F.Cu" "B.Cu") (net 1))
 	(via (at 149.5 124.5) (size 0.8) (drill 0.4) (layers "F.Cu" "B.Cu") (net 1))

Commit message: Stop hiding the hairpins behind the pads they are drawn on
The reviewer said the 135 degree bends and the odd-angle runs were still
there. They were. `route.acute_angle` skipped any corner within a pad's
*radius*, and a 0805's radius is 0.47 mm, which covers the five or six
ordinary corners a chamfered pad entry leaves inside it. Eleven of the
thirteen hairpins on these five boards sat in that shadow, because a pad
is exactly where a route that has to double back does it.

The exemption is the pad's connection point now, not a disc around it.
Two branches leaving one pad stay exempt - the pad's own copper fills the
wedge, so it is not an acid trap - but nought degrees never is: that is
one run drawn twice, and no pad excuses it.

Then the generator had to stop making them:

* `_untraced` drops the copper a second run lays on top of the first.
  The shorter is inside the longer and carries nothing it does not; both
  get trimmed, because dropping only the duplicate leaves the other
  hanging over the gap, which is `route.stub`. It runs before the runs
  are joined, while the pair is still two tracks sharing an end - once
  joined, the shared point is usually a pad, and the clean-up passes pin
  those precisely so they cannot take copper off them.
* `_straighten` only takes the direct line when it lands on the 45 grid.
  Between two pads at whatever coordinates their packages give them it
  usually does not: last round it made a nine millimetre run at 169.7
  degrees, which is the slip-of-the-mouse angle `route.odd_angle` is for.

Measured across the five boards: off-grid segments 1 to 0, 180 degree
reversals 6 to 0, and the motor board's `route.return_path` finding went
with the 11 mm of copper it was measuring.

Three corners survive, all on the FPGA board, all where a knee lands a
fraction past where its own two legs cross - legs of 0.07 and 0.25 mm on
two, 0.15 and 0.5 mm on the third. Refusing a knee that short is worse:
the segment then keeps the angle it had, a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
Routing:
- net +3V3: track 615.0 -> 626.7 mm
- net /SPI_SS: track 106.6 -> 97.4 mm
Changed lines of the file:
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@@
 	(segment (start 165.8688 103.5) (end 164.0 103.5) (width 0.2) (layer "F.Cu") (net 1))
 	(segment (start 169.1375 102.925) (end 167.6 102.925) (width 0.2) (layer "F.Cu") (net 3))
-	(segment (start 167.6 102.925) (end 166.025 104.5) (width 0.2) (layer "F.Cu") (net 3))
-	(segment (start 166.025 104.5) (end 165.519 104.5) (width 0.2) (layer "F.Cu") (net 3))
-	(segment (start 165.519 104.5) (end 169.0 104.5) (width 0.2) (layer "F.Cu") (net 3))
+	(segment (start 167.6 102.925) (end 166.812 103.712) (width 0.2) (layer "F.Cu") (net 3))
+	(segment (start 166.812 103.712) (end 166.812 104.173) (width 0.2) (layer "F.Cu") (net 3))
+	(segment (start 166.812 104.173) (end 167.139 104.5) (width 0.2) (layer "F.Cu") (net 3))
+	(segment (start 167.139 104.5) (end 169.0 104.5) (width 0.2) (layer "F.Cu") (net 3))
 	(segment (start 169.0 104.5) (end 170.5 103.0) (width 0.2) (layer "F.Cu") (net 3))
 	(segment (start 170.5 103.0) (end 170.5 96.5) (width 0.2) (layer "F.Cu") (net 3))
@@
 	(segment (start 136.1 133.905) (end 135.005 135.0) (width 0.2) (layer "F.Cu") (net 1))
 	(segment (start 135.005 135.0) (end 133.5 135.0) (width 0.2) (layer "F.Cu") (net 1))
-	(segment (start 142.475 130.095) (end 143.13 130.095) (width 0.2) (layer "F.Cu") (net 3))
-	(segment (start 143.13 130.095) (end 145.225 128.0) (width 0.2) (layer "F.Cu") (net 3))
-	(segment (start 142.475 131.365) (end 133.5 133.0) (width 0.2) (layer "F.Cu") (net 3))
+	(segment (start 142.475 130.095) (end 143.9 130.095) (width 0.2) (layer "F.Cu") (net 3))
+	(segment (start 143.9 130.095) (end 144.995 129.0) (width 0.2) (layer "F.Cu") (net 3))
+	(segment (start 144.995 129.0) (end 146.146 129.0) (width 0.2) (layer "F.Cu") (net 3))
+	(segment (start 146.146 129.0) (end 146.146 129.146) (width 0.2) (layer "F.Cu") (net 3))
+	(segment (start 146.146 129.146) (end 146.25 129.25) (width 0.2) (layer "F.Cu") (net 3))
+	(segment (start 146.25 129.25) (end 145.75 129.25) (width 0.2) (layer "F.Cu") (net 3))
+	(segment (start 145.75 129.25) (end 145.25 128.75) (width 0.2) (layer "F.Cu") (net 3))
+	(segment (start 145.25 128.75) (end 145.25 128.25) (width 0.2) (layer "F.Cu") (net 3))
+	(segment (start 145.25 128.25) (end 145.225 128.225) (width 0.2) (layer "F.Cu") (net 3))
+	(segment (start 145.225 128.225) (end 145.225 128.0) (width 0.2) (layer "F.Cu") (net 3))
+	(segment (start 142.475 131.365) (end 143.9 131.365) (width 0.2) (layer "F.Cu") (net 3))
+	(segment (start 143.9 131.365) (end 144.65 131.365) (width 0.2) (layer "F.Cu") (net 3))
+	(segment (start 144.65 131.365) (end 145.015 131.0) (width 0.2) (layer "F.Cu") (net 3))
+	(segment (start 145.015 131.0) (end 146.5 131.0) (width 0.2) (layer "F.Cu") (net 3))
+	(segment (start 146.5 131.0) (end 147.125 130.375) (width 0.2) (layer "F.Cu") (net 3))
+	(segment (start 147.125 130.375) (end 147.125 130.009) (width 0.2) (layer "F.Cu") (net 3))
+	(segment (start 147.125 130.009) (end 146.866 129.75) (width 0.2) (layer "F.Cu") (net 3))
+	(segment (start 146.866 129.75) (end 142.75 129.75) (width 0.2) (layer "F.Cu") (net 3))
+	(segment (start 142.75 129.75) (end 139.5 133.0) (width 0.2) (layer "F.Cu") (net 3))
+	(segment (start 139.5 133.0) (end 133.5 133.0) (width 0.2) (layer "F.Cu") (net 3))
 	(segment (start 142.475 132.635) (end 143.9 132.635) (width 0.2) (layer "F.Cu") (net 16))
 	(segment (start 143.9 132.635) (end 144.65 132.635) (width 0.2) (layer "F.Cu") (net 16))
@@
 	(segment (start 125.5 79.75) (end 127.5 81.75) (width 0.2) (layer "F.Cu") (net 3))
 	(segment (start 127.5 81.75) (end 127.5 81.825) (width 0.2) (layer "F.Cu") (net 3))
-	(segment (start 127.5 81.825) (end 127.675 82.0) (width 0.2) (layer "F.Cu") (net 3))
-	(segment (start 127.675 82.0) (end 127.675 81.825) (width 0.2) (layer "F.Cu") (net 3))
+	(segment (start 127.5 81.825) (end 127.5875 81.9125) (width 0.2) (layer "F.Cu") (net 3))
+	(segment (start 127.5875 81.9125) (end 127.675 81.825) (width 0.2) (layer "F.Cu") (net 3))
 	(segment (start 127.675 81.825) (end 127.75 81.75) (width 0.2) (layer "F.Cu") (net 3))
 	(segment (start 127.75 81.75) (end 127.75 81.25) (width 0.2) (layer "F.Cu") (net 3))
@@
 	(segment (start 148.0 136.25) (end 158.25 126.0) (width 0.2) (layer "F.Cu") (net 19))
 	(segment (start 158.25 126.0) (end 174.0 126.0) (width 0.2) (layer "F.Cu") (net 19))
-	(segment (start 174.0 126.0) (end 164.75 126.0) (width 0.2) (layer "F.Cu") (net 19))
 	(segment (start 164.75 126.0) (end 157.0 133.75) (width 0.2) (layer "F.Cu") (net 19))
 	(segment (start 157.0 133.75) (end 157.0 133.825) (width 0.2) (layer "F.Cu") (net 19))

Commit message: Reroute the FPGA board and record what the rip-up loop bought
Eleven rip-ups and three re-orderings later, and the sixth promotion rolled
back because it left I2S_SCK with no lane:

  route.detour   VCCPLL at 5.0x   ->  gone
  route.wander   4 runs           ->  2
  acute corners  3                ->  2
  route.return_path 7 nets        ->  6
  DRC errors     1 unconnected    ->  0

Board findings 1/10/8 -> 0/9/8, and the gate goes from 5 blocking to 3. Under
KiCad's own checks the board is now clean: no DRC errors, nothing unconnected,
no schematic-parity findings.

What is left is the two-layer choice itself. Six nets run over cuts in the
back-side plane because a 48-pin QFN with no inner layer has to bring the SPI
bus out somewhere, and re-ordering cannot make a plane that is not there.
Recorded in REVIEW.md rather than waived.

All thirty example images are re-rendered. 514 tests pass on KiCad 10.0.4 and
9.0.9; ruff clean.

Co-Authored-By: Claude Opus 5 <noreply@anthropic.com>
Claude-Session: https://claude.ai/code/session_01DUj7Ltu92tWg159mCSacwY
Routing:
- net /VCCPLL: track 113.9 -> 25.5 mm, vias 4 -> 0
- net +3V3: track 626.7 -> 685.4 mm, vias 12 -> 14
- net /OUTR: track 66.0 -> 20.6 mm, vias 4 -> 0
- net /SPI_SCK: track 79.1 -> 115.9 mm, vias 4 -> 2
- net /SPI_SO: track 122.3 -> 96.7 mm
- net /SPI_SI: track 86.4 -> 73.2 mm, vias 8 -> 6
- net /OUTL: track 27.2 -> 40.2 mm, vias 4 -> 2
- net /VNEG: track 18.5 -> 30.8 mm, vias 0 -> 2
- net /CRESET: track 141.8 -> 146.0 mm, vias 6 -> 4
- net GND: track 134.2 -> 138.1 mm, vias 170 -> 177
- net /+1V2: track 115.1 -> 112.4 mm
- net /LDOO: track 19.0 -> 16.5 mm, vias 0 -> 2
- net /CLK12: track 38.1 -> 40.5 mm, vias 2 -> 0
- net /SPI_SS: track 97.4 -> 95.1 mm, vias 2 -> 6
- net /CAPP: track 16.6 -> 15.4 mm, vias 2 -> 0
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