File: examples/fpga-audio/reviewed/fpga-audio.kicad_sch (KiCad schematic)
At the start: 26 parts, among them J1 3V3 IN, J2 AUDIO OUT, J3 SPI PROG, U1 iCE40UP5K, U2 PCM5102A, U3 AP2112K-1.2, U4 W25Q32JV, X1 12MHz

Commit message: Show the fifth example, and say what the five of them agree on
Six renders of the iCE40 board and the section that goes with them, plus two
last fixes of my own: the sheet is A3, because four units of one symbol and
twenty parts do not fit on A4 and 177 items were sitting off the page; and GND
carries a PWR_FLAG, because every ground pin on this board is a power *input*
and ERC was right to say so.

The README now ends with what the set says together rather than what each
board says on its own. Three findings appear on every board with a fine-pitch
part - TSSOP-16, SOT-23-5 and QFN-48, three package sizes apart - and all of
them trace to the escape from the package eating the distance budget before
any component can be placed. Two more are blind spots approached from opposite
directions: the rules can tell a supply net from a signal, and cannot tell a
supply this board makes from one it is handed.

And two things no rule catches at all, both visible in the plots: every
connection on these schematics is a label rather than a wire, and the routing
looks autorouted because it is.
Changed lines of the file:
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@@
 (kicad_sch (version 20250114) (generator "eda-toolkit") (generator_version "9.0")
-  (paper "A4")
+  (paper "A3")
   (title_block
   	(title "iCE40UP5K to PCM5102A, I2S out")
@@
     (instances (project "fpga-audio" (path "/434dea94-d96f-5288-b60c-67317d440f4e" (reference "C15") (unit 1))))
   )
-  (wire (pts (xy 50.800000000000004 59.69) (xy 50.800000000000004 62.23)) (stroke (width 0) (type default)) (uuid "37d1d27a-0d34-54c7-85f0-6bfddc0b4157-w"))
-  (label "+3V3" (at 50.800000000000004 62.23 0) (effects (font (size 1.27 1.27)) (justify left bottom)) (uuid "37d1d27a-0d34-54c7-85f0-6bfddc0b4157-l"))
-  (symbol (lib_id "power:PWR_FLAG") (at 50.800000000000004 59.69 0) (unit 1)
-    (exclude_from_sim no) (in_bom no) (on_board yes) (dnp no)
-    (property "Reference" "#FLG01" (at 50.800000000000004 59.69 0) (effects (font (size 1.27 1.27)) hide))
-    (property "Value" "PWR_FLAG" (at 50.800000000000004 55.879999999999995 0) (effects (font (size 1.27 1.27))))
-    (property "Footprint" "" (at 50.800000000000004 59.69 0) (effects (font (size 1.27 1.27)) hide))
-    (property "Datasheet" "" (at 50.800000000000004 59.69 0) (effects (font (size 1.27 1.27)) hide))
+  (wire (pts (xy 165.10000000000002 30.48) (xy 165.10000000000002 33.02)) (stroke (width 0) (type default)) (uuid "37d1d27a-0d34-54c7-85f0-6bfddc0b4157-w"))
+  (label "+3V3" (at 165.10000000000002 33.02 0) (effects (font (size 1.27 1.27)) (justify left bottom)) (uuid "37d1d27a-0d34-54c7-85f0-6bfddc0b4157-l"))
+  (symbol (lib_id "power:PWR_FLAG") (at 165.10000000000002 30.48 0) (unit 1)
+    (exclude_from_sim no) (in_bom no) (on_board yes) (dnp no)
+    (property "Reference" "#FLG01" (at 165.10000000000002 30.48 0) (effects (font (size 1.27 1.27)) hide))
+    (property "Value" "PWR_FLAG" (at 165.10000000000002 26.67 0) (effects (font (size 1.27 1.27))))
+    (property "Footprint" "" (at 165.10000000000002 30.48 0) (effects (font (size 1.27 1.27)) hide))
+    (property "Datasheet" "" (at 165.10000000000002 30.48 0) (effects (font (size 1.27 1.27)) hide))
     (pin "1" (uuid "37d1d27a-0d34-54c7-85f0-6bfddc0b4157-p"))
     (instances (project "fpga-audio" (path "/434dea94-d96f-5288-b60c-67317d440f4e" (reference "#FLG01") (unit 1))))
   )
-  (text "A 0.5 mm pitch QFN with pads on four sides is not a two layer board." (at 18.0 25.08 0) (effects (font (size 1.27 1.27)) (justify left top)))
-  (text "A real iCE40 design drops each pin into an inner layer; this one has" (at 18.0 30.16 0) (effects (font (size 1.27 1.27)) (justify left top)))
-  (text "no inner layer, so all 48 escape on the top at 0.2 mm track and" (at 18.0 35.24 0) (effects (font (size 1.27 1.27)) (justify left top)))
-  (text "0.2 mm clearance - a fine-line process, and the reason a 7 mm chip" (at 18.0 40.32 0) (effects (font (size 1.27 1.27)) (justify left top)))
-  (text "needs 25 mm of board around it before anything else can be placed." (at 18.0 45.4 0) (effects (font (size 1.27 1.27)) (justify left top)))
-  (text "Two rails: 3.3 V in for the I/O banks, the codec and the flash, and" (at 18.0 50.48 0) (effects (font (size 1.27 1.27)) (justify left top)))
-  (text "1.2 V from U3 for the core, with C15 and C5 on the two VCC pins and" (at 18.0 55.56 0) (effects (font (size 1.27 1.27)) (justify left top)))
-  (text "on VCCPLL - which the datasheet would rather see filtered from the" (at 18.0 60.64 0) (effects (font (size 1.27 1.27)) (justify left top)))
-  (text "core rail than tied straight to it, and is a thing this board is" (at 18.0 65.72 0) (effects (font (size 1.27 1.27)) (justify left top)))
-  (text "not doing." (at 18.0 70.8 0) (effects (font (size 1.27 1.27)) (justify left top)))
-  (text "U1 boots from U4 over its own SPI port; J3 is that bus plus CRESET," (at 18.0 75.88 0) (effects (font (size 1.27 1.27)) (justify left top)))
-  (text "so the flash can be written in circuit. R1 and R2 hold CRESET and" (at 18.0 80.96 0) (effects (font (size 1.27 1.27)) (justify left top)))
-  (text "CDONE up, both being open drain." (at 18.0 86.04 0) (effects (font (size 1.27 1.27)) (justify left top)))
-  (text "U2's mode pins are strapped to a rail rather than driven: 16-bit" (at 18.0 91.12 0) (effects (font (size 1.27 1.27)) (justify left top)))
-  (text "I2S, no de-emphasis, normal filter, un-muted." (at 18.0 96.2 0) (effects (font (size 1.27 1.27)) (justify left top)))
+  (wire (pts (xy 180.34 30.48) (xy 180.34 33.02)) (stroke (width 0) (type default)) (uuid "e2763eba-a7fb-5ace-a986-8da7cb63b565-w"))
+  (label "GND" (at 180.34 33.02 0) (effects (font (size 1.27 1.27)) (justify left bottom)) (uuid "e2763eba-a7fb-5ace-a986-8da7cb63b565-l"))
+  (symbol (lib_id "power:PWR_FLAG") (at 180.34 30.48 0) (unit 1)
+    (exclude_from_sim no) (in_bom no) (on_board yes) (dnp no)
+    (property "Reference" "#FLG02" (at 180.34 30.48 0) (effects (font (size 1.27 1.27)) hide))
+    (property "Value" "PWR_FLAG" (at 180.34 26.67 0) (effects (font (size 1.27 1.27))))
+    (property "Footprint" "" (at 180.34 30.48 0) (effects (font (size 1.27 1.27)) hide))
+    (property "Datasheet" "" (at 180.34 30.48 0) (effects (font (size 1.27 1.27)) hide))
+    (pin "1" (uuid "e2763eba-a7fb-5ace-a986-8da7cb63b565-p"))
+    (instances (project "fpga-audio" (path "/434dea94-d96f-5288-b60c-67317d440f4e" (reference "#FLG02") (unit 1))))
+  )
+  (text "A 0.5 mm pitch QFN with pads on four sides is not a two layer board." (at 18.0 27.08 0) (effects (font (size 1.27 1.27)) (justify left top)))
+  (text "A real iCE40 design drops each pin into an inner layer; this one has" (at 18.0 32.16 0) (effects (font (size 1.27 1.27)) (justify left top)))
+  (text "no inner layer, so all 48 escape on the top at 0.2 mm track and" (at 18.0 37.24 0) (effects (font (size 1.27 1.27)) (justify left top)))
+  (text "0.2 mm clearance - a fine-line process, and the reason a 7 mm chip" (at 18.0 42.32 0) (effects (font (size 1.27 1.27)) (justify left top)))
+  (text "needs 25 mm of board around it before anything else can be placed." (at 18.0 47.4 0) (effects (font (size 1.27 1.27)) (justify left top)))
+  (text "Two rails: 3.3 V in for the I/O banks, the codec and the flash, and" (at 18.0 52.48 0) (effects (font (size 1.27 1.27)) (justify left top)))
+  (text "1.2 V from U3 for the core, with C15 and C5 on the two VCC pins and" (at 18.0 57.56 0) (effects (font (size 1.27 1.27)) (justify left top)))
+  (text "on VCCPLL - which the datasheet would rather see filtered from the" (at 18.0 62.64 0) (effects (font (size 1.27 1.27)) (justify left top)))
+  (text "core rail than tied straight to it, and is a thing this board is" (at 18.0 67.72 0) (effects (font (size 1.27 1.27)) (justify left top)))
+  (text "not doing." (at 18.0 72.8 0) (effects (font (size 1.27 1.27)) (justify left top)))
+  (text "U1 boots from U4 over its own SPI port; J3 is that bus plus CRESET," (at 18.0 77.88 0) (effects (font (size 1.27 1.27)) (justify left top)))
+  (text "so the flash can be written in circuit. R1 and R2 hold CRESET and" (at 18.0 82.96 0) (effects (font (size 1.27 1.27)) (justify left top)))
+  (text "CDONE up, both being open drain." (at 18.0 88.04 0) (effects (font (size 1.27 1.27)) (justify left top)))
+  (text "U2's mode pins are strapped to a rail rather than driven: 16-bit" (at 18.0 93.12 0) (effects (font (size 1.27 1.27)) (justify left top)))
+  (text "I2S, no de-emphasis, normal filter, un-muted." (at 18.0 98.2 0) (effects (font (size 1.27 1.27)) (justify left top)))
   (sheet_instances
     (path "/" (page "1"))

Commit message: Read the five as an engineer would, and make the toolkit act on it
examples/REVIEW.md is the pass: the five designs read for circuit theory,
layout physics and readability, every finding dispatched to one of four
places - a rule, a fix, a reasoned waiver, or named as open. The headline
result: every reviewed/ project now PASSES its own gate, every as-generated/
still fails it, and every waiver is an engineering argument a reviewer can
disagree with.

Four new rules, each calibrated against KiCad's 18 human-drawn demo projects:

* readability.label_only - the sheet connects by name, not by wire; the
  single most recognisable mark of a generated schematic. 0 findings on the
  human corpus, 71-100% on ours.
* analog.no_dc_path - a net of only capacitors and connectors has nothing
  setting its DC level. Found a real fault: the op-amp filter's AC-coupled
  output floated. 0 findings on the corpus.
* route.detour - routed copper against the MST of the net's pads; the scenic
  tour an autorouter takes. 8 human boards fired at 2.5x, 0 at the shipped 4x.
* route.return_path - signal running over cuts in the other layer's ground
  fill, computed from the difference between a zone's outline and its fill,
  which the parser now keeps. Fires on 4 real demo boards, because real
  two-layer boards genuinely have the disease.

Three rules re-judged on evidence instead of names:

* analog.missing_decoupling reads pin electrical types: only power_in pins
  ask for a capacitor, and a net an output pin drives is never asked - a cap
  on an op-amp output is somebody's control loop. Retires the VBUS/VREF
  false positives without a single waiver.
* track.thin_power measures the longest contiguous narrow run against a
  power_neck_mm allowance. Pad entries and fine-pitch escapes pass; thin
  trunks still fail. 9 demo boards fired before, 0 after - all nine were necks.
* net.single_pin honours no-connect flags: a flagged pin is a decision.

And the designs themselves got the fixes the pa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
Parts:
- added C17: 10u, Capacitor_SMD:C_0603_1608Metric, symbol Device:C
- added R3: 100R, Resistor_SMD:R_0603_1608Metric, symbol Device:R
- added R4: 10k, Resistor_SMD:R_0603_1608Metric, symbol Device:R
- C12: value 1u -> 2u2; MPN CL10A105KB8NNNC -> CL10A225KO8NNNC
Connections:
- net +1V2: now also R3.1; no longer C5.1, U1.29 (VCCPLL)
- net +3V3: now also R4.1
- net CAPM: now also C13.2; no longer C14.1
- net GND: now also C14.2, C17.2; no longer C13.2
- net SPI_SS: now also R4.2
- net VNEG: now also C14.1; no longer C14.2
- new net VCCPLL: C17.1, C5.1, R3.2, U1.29 (VCCPLL)
- no-connect marks 30 -> 31
Other:
- note added: "1.2 V from U3 for the core, with C15 on the VCC pins. VCCPLL is"
- note added: "R4 holds the flash chip select up while the FPGA is still"
- note added: "configuring and its pins are floating."
- note added: "filtered from the core rail through R3 with C17 and C5 at the pin,"
- note added: "which is what keeps core switching noise out of the PLL."
- note removed: "1.2 V from U3 for the core, with C15 and C5 on the two VCC pins and"
- note removed: "core rail than tied straight to it, and is a thing this board is"
- note removed: "not doing."
- note removed: "on VCCPLL - which the datasheet would rather see filtered from the"
