File: examples/fpga-audio/reviewed/fpga-audio.kicad_sch (KiCad schematic)
At the start: 29 parts, among them J1 3V3 IN, J2 AUDIO OUT, J3 SPI PROG, U1 iCE40UP5K, U2 PCM5102A, U3 AP2112K-1.2, U4 W25Q32JV, X1 12MHz

Commit message: Route the sheets, and anchor the ground vias where the loop is
The user's verdict on the last round stood: none of the five schematics
read as a human drawing, and the artwork still had its physics wrong.
This round answers both.

The schematic side replaces the stub-and-label sheet with a router.
Every signal net becomes a tree of straight, L-, Z- and detour-shaped
runs on the 1.27 mm grid: legs leave a pin along its own stub, escape
distances stagger so a bus does not fight over one column, every pin
reserves a runway another wire may cross but not ride along, and the
sheet frame, title block and notes are obstacles like any symbol.
Fragments merge Kruskal-style so a rail whose regulator is boxed in
still gets its capacitors chained; each surviving fragment keeps one
label, because the label is what names the net. Collinear same-net
segments are unioned and then split at every tee - KiCad 9's
connectivity requires files drawn the way the editor draws them, with
a junction dot and a wire break wherever a branch tees in, and a wire
that runs through a junction connects on one side of it only. That
last fact cost an evening and is now a comment.

Trying to draw the wires found what no rule had: the buck's LED was
upside down with its ground pointing up into the resistor above it,
both breakout headers faced away from everything they connect to
(fixed with mirrored symbols, which Part now supports), the FPGA
sheet's notes printed over the 1.2 V regulator, and its programming
header sat inside the title block. Wired: buck, motor and op-amp
completely; the Pico carrier 31 of 33 nets; the FPGA board 16 of 19 -
what stays labelled is what a human would label too.

The artwork side anchors every FPGA decoupling capacitor's ground via
against its own pad, on the far side from the supply pad, with the
1.2 mm stub as the whole loop - retiring all seven
layout.decoupling_via findings and that waiver with them. A back_cost
experiment (0.4 to 0.6) to shrink the return-path cuts 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
Other:
- moved on the sheet: J3
