File: examples/fpga-audio/reviewed/fpga-audio.kicad_sch (KiCad schematic)
At the start: 36 parts, among them J1 3V3 IN, J2 AUDIO OUT, J3 SPI PROG, U1 iCE40UP5K, U2 PCM5102A, U3 AP2112K-1.2, U4 W25Q32JV, X1 12MHz

Commit message: Rebuild golden layouts and gate floorplan quality
Connections:
- net CRESET: now also J3.3 (Pin_3); no longer J3.5 (Pin_5)
- net GND: now also J2.3 (Pin_3); no longer J2.2 (Pin_2)
- net OUTL: now also J2.2 (Pin_2); no longer J2.3 (Pin_3)
- net SPI_SCK: now also J3.4 (Pin_4); no longer J3.2 (Pin_2)
- net SPI_SI: now also J3.5 (Pin_5); no longer J3.3 (Pin_3)
- net SPI_SO: now also J3.2 (Pin_2); no longer J3.4 (Pin_4)
Other:
- note added: "Its 0.2 mm top escape spreads to 0.8 mm before routing; bottom"
- note added: "The 0.5 mm QFN uses a four-layer stack: outer signal layers,"
- note added: "an uninterrupted In1 ground plane and a +3V3 In2 power plane."
- note added: "signal hops no longer cut the reference plane beneath it."
- note removed: "0.2 mm track and 0.2 mm clearance - a fine-line process, and"
- note removed: "A 0.5 mm pitch QFN with pads on four sides is not a two layer"
- note removed: "board. A real iCE40 design drops each pin into an inner layer;"
- note removed: "the reason a 7 mm chip needs 25 mm of board around it."
- note removed: "this one has no inner layer, so all 48 escape on the top at"
Changed lines of the file:
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@@
   (paper "A3")
   (title_block
-  	(title "iCE40UP5K to PCM5102A, I2S out")
-  	(date "2026-08-12")
-  	(rev "A")
-  	(company "kicad_skills examples")
-  	(comment 1 "generated 2026-08-12 by Claude Code (claude-fable-5)")
-  	(comment 2 "from tools/make_examples.py in sabas0ba/kicad_skills")
+    (title "iCE40UP5K to PCM5102A, I2S out")
+    (date "2026-09-05")
+    (rev "A")
+    (company "kicad_skills examples")
+    (comment 1 "generated 2026-09-05 by OpenAI Codex")
+    (comment 2 "from tools/make_examples.py in sabas0ba/kicad_skills")
   )
   (wire (pts (xy 349.25 123.19) (xy 351.79 123.19)) (stroke (width 0) (type default)))
@@
   (wire (pts (xy 396.24 102.87) (xy 396.24 107.95)) (stroke (width 0) (type default)))
   (wire (pts (xy 349.25 100.33) (xy 397.51 100.33)) (stroke (width 0) (type default)))
-  (wire (pts (xy 397.51 100.33) (xy 397.51 113.03)) (stroke (width 0) (type default)))
-  (wire (pts (xy 396.24 113.03) (xy 397.51 113.03)) (stroke (width 0) (type default)))
+  (wire (pts (xy 397.51 100.33) (xy 397.51 110.49)) (stroke (width 0) (type default)))
+  (wire (pts (xy 396.24 110.49) (xy 397.51 110.49)) (stroke (width 0) (type default)))
   (wire (pts (xy 349.25 107.95) (xy 350.52 107.95)) (stroke (width 0) (type default)))
   (wire (pts (xy 350.52 107.95) (xy 350.52 151.13)) (stroke (width 0) (type default)))
@@
   (wire (pts (xy 176.53 166.37) (xy 176.53 181.61)) (stroke (width 0) (type default)))
   (wire (pts (xy 176.53 166.37) (xy 257.81 166.37)) (stroke (width 0) (type default)))
-  (wire (pts (xy 257.81 166.37) (xy 257.81 245.11)) (stroke (width 0) (type default)))
-  (wire (pts (xy 257.81 245.11) (xy 260.35 245.11)) (stroke (width 0) (type default)))
+  (wire (pts (xy 257.81 166.37) (xy 257.81 240.03)) (stroke (width 0) (type default)))
+  (wire (pts (xy 257.81 240.03) (xy 260.35 240.03)) (stroke (width 0) (type default)))
   (junction (at 66.04 36.83) (diameter 0) (color 0 0 0 0))
   (junction (at 163.83 41.91) (diameter 0) (color 0 0 0 0))
@@
   (label "OUTR" (at 396.24 107.95 0) (effects (font (size 1.27 1.27)) (justify left bottom)))
   (wire (pts (xy 393.7 110.49) (xy 396.24 110.49)) (stroke (width 0) (type default)))
+  (label "OUTL" (at 396.24 110.49 0) (effects (font (size 1.27 1.27)) (justify left bottom)))
   (wire (pts (xy 393.7 113.03) (xy 396.24 113.03)) (stroke (width 0) (type default)))
-  (label "OUTL" (at 396.24 113.03 0) (effects (font (size 1.27 1.27)) (justify left bottom)))
   (symbol (lib_id "Connector:Conn_01x03_Pin") (at 388.62 110.49 0.0) (unit 1)
     (exclude_from_sim no) (in_bom yes) (on_board yes) (dnp no)
@@
   (label "SPI_SS" (at 260.35 234.95 0) (effects (font (size 1.27 1.27)) (justify right bottom)))
   (wire (pts (xy 262.89 237.49) (xy 260.35 237.49)) (stroke (width 0) (type default)))
-  (label "SPI_SCK" (at 260.35 237.49 0) (effects (font (size 1.27 1.27)) (justify right bottom)))
+  (label "SPI_SO" (at 260.35 237.49 0) (effects (font (size 1.27 1.27)) (justify right bottom)))
   (wire (pts (xy 262.89 240.03) (xy 260.35 240.03)) (stroke (width 0) (type default)))
-  (label "SPI_SI" (at 260.35 240.03 0) (effects (font (size 1.27 1.27)) (justify right bottom)))
+  (label "CRESET" (at 260.35 240.03 0) (effects (font (size 1.27 1.27)) (justify right bottom)))
   (wire (pts (xy 262.89 242.57) (xy 260.35 242.57)) (stroke (width 0) (type default)))
-  (label "SPI_SO" (at 260.35 242.57 0) (effects (font (size 1.27 1.27)) (justify right bottom)))
+  (label "SPI_SCK" (at 260.35 242.57 0) (effects (font (size 1.27 1.27)) (justify right bottom)))
   (wire (pts (xy 262.89 245.11) (xy 260.35 245.11)) (stroke (width 0) (type default)))
-  (label "CRESET" (at 260.35 245.11 0) (effects (font (size 1.27 1.27)) (justify right bottom)))
+  (label "SPI_SI" (at 260.35 245.11 0) (effects (font (size 1.27 1.27)) (justify right bottom)))
   (wire (pts (xy 262.89 247.65) (xy 260.35 247.65)) (stroke (width 0) (type default)))
   (symbol (lib_id "Connector:Conn_01x06_Pin") (at 267.97 240.03 0.0) (mirror y) (unit 1)
@@
   (wire (pts (xy 24.13 41.91) (xy 24.13 49.53)) (stroke (width 0) (type default)))
   (wire (pts (xy 24.13 49.53) (xy 29.21 49.53)) (stroke (width 0) (type default)))
-  (wire (pts (xy 396.24 110.49) (xy 403.86 110.49)) (stroke (width 0) (type default)))
-  (wire (pts (xy 403.86 110.49) (xy 403.86 118.11)) (stroke (width 0) (type default)))
+  (wire (pts (xy 396.24 113.03) (xy 403.86 113.03)) (stroke (width 0) (type default)))
+  (wire (pts (xy 403.86 113.03) (xy 403.86 118.11)) (stroke (width 0) (type default)))
   (wire (pts (xy 260.35 247.65) (xy 252.73 247.65)) (stroke (width 0) (type default)))
   (wire (pts (xy 252.73 247.65) (xy 252.73 252.73)) (stroke (width 0) (type default)))
@@
   (junction (at 38.1 36.83) (diameter 0) (color 0 0 0 0))
   (junction (at 175.26 260.35) (diameter 0) (color 0 0 0 0))
-  (text "A 0.5 mm pitch QFN with pads on four sides is not a two layer" (at 17.78 232.0 0) (effects (font (size 1.27 1.27)) (justify left top)))
-  (text "board. A real iCE40 design drops each pin into an inner layer;" (at 17.78 236.0 0) (effects (font (size 1.27 1.27)) (justify left top)))
-  (text "this one has no inner layer, so all 48 escape on the top at" (at 17.78 240.0 0) (effects (font (size 1.27 1.27)) (justify left top)))
-  (text "0.2 mm track and 0.2 mm clearance - a fine-line process, and" (at 17.78 244.0 0) (effects (font (size 1.27 1.27)) (justify left top)))
-  (text "the reason a 7 mm chip needs 25 mm of board around it." (at 17.78 248.0 0) (effects (font (size 1.27 1.27)) (justify left top)))
+  (text "The 0.5 mm QFN uses a four-layer stack: outer signal layers," (at 17.78 232.0 0) (effects (font (size 1.27 1.27)) (justify left top)))
+  (text "an uninterrupted In1 ground plane and a +3V3 In2 power plane." (at 17.78 236.0 0) (effects (font (size 1.27 1.27)) (justify left top)))
+  (text "Its 0.2 mm top escape spreads to 0.8 mm before routing; bottom" (at 17.78 240.0 0) (effects (font (size 1.27 1.27)) (justify left top)))
+  (text "signal hops no longer cut the reference plane beneath it." (at 17.78 244.0 0) (effects (font (size 1.27 1.27)) (justify left top)))
   (text "C1 10u + C2 100n: the 3.3 V input, at U3." (at 100.0 78.0 0) (effects (font (size 1.27 1.27)) (justify left top)))
   (text "C3/C4: the 1.2 V core rail it makes. C15 sits" (at 100.0 82.0 0) (effects (font (size 1.27 1.27)) (justify left top)))
