File: examples/fpga-audio/reviewed/fpga-audio.kicad_sch (KiCad schematic)
At the start: 36 parts, among them J1 3V3 IN, J2 AUDIO OUT, J3 SPI PROG, U1 iCE40UP5K, U2 PCM5102A, U3 AP2112K-1.2, U4 W25Q32JV, X1 12MHz

Commit message: feat(examples): the FPGA board on two layers, and the rim fenced in the generator
The last of the five, and the one that had to be re-floorplanned rather than
converted: a 48-pin QFN, a codec, a boot flash and an oscillator escaped on two
faces. All five examples are now two-layer and gate clean.

What moved, and why:

* the boot flash came up ten millimetres to meet the FPGA's SPI port, the
  configuration header eight west along the bottom edge it serves, and CRESET's
  pull-up now stands between its two ends instead of beside CDONE's. Together
  those took `layout.connection_span` from nine findings - worst 51.5 mm - to
  the four I2S runs at 25.7 mm, which are the two packages' own width.
* the outer ring of the pour is now a router keepout, not just something the
  review reports afterwards. On the widest board in the set the perimeter is
  the emptiest lane there is and the router took it twice, for 20.5 mm of the
  bottom edge and 11.5 mm of the right. Reporting that is `layout.pour_edge_cut`;
  not building it is the generator's job.
* the input rail goes round the screw terminal rather than under its body, the
  core rail's link to its spine is asked for at the width it lands on, and the
  oscillator's bypass takes its supply from the neighbour eight millimetres
  away instead of the flash's bypass fifty-two millimetres away.

What is judged rather than fixed is in `gate.toml` with its measurements: the
two-layer return path on the SPI bus, XSMT's detour - R6 in the corridor was
tried and left five nets with no lane at all - the I2S spans, and two marginal
router artifacts on one escape.

Co-Authored-By: Claude Opus 5 <noreply@anthropic.com>
Claude-Session: https://claude.ai/code/session_01XQE7UkE9WTSMW3oZ3kLeCt
Parts:
- added D3: SMAJ5.0A, Diode_SMD:D_SMA, symbol Device:D_Zener
- added F1: 500mA, Fuse:Fuse_1206_3216Metric, symbol Device:Fuse
- added R5: 33R, Resistor_SMD:R_0603_1608Metric, symbol Device:R
- added R6: 10k, Resistor_SMD:R_0603_1608Metric, symbol Device:R
Connections:
- net +3V3: now also D3.1 (K), F1.2; no longer J1.1 (Pin_1), U2.17 (XSMT)
- net CLK12: now also R5.2; no longer X1.3 (OUT)
- net CRESET: now also J3.5 (Pin_5); no longer J3.3 (Pin_3)
- net GND: now also J2.2 (Pin_2), D3.2 (A), R6.2; no longer J2.3 (Pin_3)
- net OUTL: now also J2.3 (Pin_3); no longer J2.2 (Pin_2)
- net SPI_SCK: now also J3.2 (Pin_2); no longer J3.4 (Pin_4)
- net SPI_SI: now also J3.3 (Pin_3); no longer J3.5 (Pin_5)
- net SPI_SO: now also J3.4 (Pin_4); no longer J3.2 (Pin_2)
- net XSMT: now reaches U1.31 (IOT_42b)
- net XSMT: now also U2.17 (XSMT), R6.1
- new net OSC_OUT: R5.1, X1.3 (OUT)
- new net VIN: F1.1, J1.1 (Pin_1)
- no-connect marks 31 -> 30
Other:
- note added: "0.2 mm track and 0.2 mm clearance - a fine-line process, and"
- note added: "A 0.5 mm pitch QFN with pads on four sides is not a two layer"
- note added: "C11/C16 bypass its supplies; C12-C14 are the charge"
- note added: "F1 500 mA and D3 (5 V standoff) guard the input:"
- note added: "R5 33R at X1's output damps the 12 MHz edge into"
- note added: "R6 holds it low so the DAC comes up muted, and the"
- note added: "board. A real iCE40 design drops each pin into an inner layer;"
- note added: "configured FPGA un-mutes it - no power-up pop."
- note added: "no de-emphasis, normal filter. XSMT is the exception:"
- note added: "not hold the rail under the FPGA's 3.6 V maximum."
- note added: "pump and LDO reservoirs the datasheet asks for."
- note added: "reversed leads flow through D3 and open F1. D3 does"
- note added: "the 30 mm run to the FPGA: the clock arrives once."
- note added: "the reason a 7 mm chip needs 25 mm of board around it."
- note added: "this one has no inner layer, so all 48 escape on the top at"
- note removed: "Its 0.2 mm top escape spreads to 0.8 mm before routing; bottom"
- note removed: "The 0.5 mm QFN uses a four-layer stack: outer signal layers,"
- note removed: "an uninterrupted In1 ground plane and a +3V3 In2 power plane."
- note removed: "and LDO reservoirs the datasheet asks for."
- note removed: "bypass its supplies; C12-C14 are the charge pump"
- note removed: "no de-emphasis, normal filter, un-muted. C11/C16"
- note removed: "signal hops no longer cut the reference plane beneath it."
- moved on the sheet: C3, C4, C9, J1, U3
