File: examples/opamp-filter/reviewed/opamp-filter.kicad_pcb (KiCad board)
At the start: 2 copper layers, 80 x 45 mm, 17 parts, among them J1 IN, J2 5V, J3 OUT, U1 MCP6001R, U2 MCP6001R

Commit message: Read the five as an engineer would, and make the toolkit act on it
examples/REVIEW.md is the pass: the five designs read for circuit theory,
layout physics and readability, every finding dispatched to one of four
places - a rule, a fix, a reasoned waiver, or named as open. The headline
result: every reviewed/ project now PASSES its own gate, every as-generated/
still fails it, and every waiver is an engineering argument a reviewer can
disagree with.

Four new rules, each calibrated against KiCad's 18 human-drawn demo projects:

* readability.label_only - the sheet connects by name, not by wire; the
  single most recognisable mark of a generated schematic. 0 findings on the
  human corpus, 71-100% on ours.
* analog.no_dc_path - a net of only capacitors and connectors has nothing
  setting its DC level. Found a real fault: the op-amp filter's AC-coupled
  output floated. 0 findings on the corpus.
* route.detour - routed copper against the MST of the net's pads; the scenic
  tour an autorouter takes. 8 human boards fired at 2.5x, 0 at the shipped 4x.
* route.return_path - signal running over cuts in the other layer's ground
  fill, computed from the difference between a zone's outline and its fill,
  which the parser now keeps. Fires on 4 real demo boards, because real
  two-layer boards genuinely have the disease.

Three rules re-judged on evidence instead of names:

* analog.missing_decoupling reads pin electrical types: only power_in pins
  ask for a capacitor, and a net an output pin drives is never asked - a cap
  on an op-amp output is somebody's control loop. Retires the VBUS/VREF
  false positives without a single waiver.
* track.thin_power measures the longest contiguous narrow run against a
  power_neck_mm allowance. Pad entries and fine-pitch escapes pass; thin
  trunks still fail. 9 demo boards fired before, 0 after - all nine were necks.
* net.single_pin honours no-connect flags: a flagged pin is a decision.

And the designs themselves got the fixes the pa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
Parts:
- added R6: 100k, Resistor_SMD:R_0805_2012Metric, F.Cu at (170.0, 87.0)
- added R7: 100k, Resistor_SMD:R_0805_2012Metric, F.Cu at (112.0, 86.0)
Routing:
- net /OUT_AC: track 12.4 -> 25.7 mm
- net /IN: track 8.42 -> 20.1 mm
- net GND: track 54.8 -> 65.8 mm, vias 9 -> 11
