File: examples/opamp-filter/reviewed/opamp-filter.kicad_sch (KiCad schematic)
At the start: 29 parts, among them J1 IN, J2 5V, J3 OUT, U1 MCP6001R, U2 MCP6001R

Commit message: feat(examples): rebuild the opamp-filter layout along its signal row
The filter is drawn as one straight row from input to output with each part's
tap a stated spur; the supply crosses under the row once, through stated vias,
instead of running round the board's edge; the reference block sits under the
part it feeds. 58x42 -> 54x38 mm and 376 -> 255 mm of track. Connector pin
legends sit on their own pins.

Co-Authored-By: Claude Opus 5.5 <noreply@anthropic.com>
Claude-Session: https://claude.ai/code/session_013K3aKVeLLeg21eHKEw4dQ7
Parts:
- added H3: M3, MountingHole:MountingHole_3.2mm_M3, symbol Mechanical:MountingHole
Other:
- moved on the sheet: FID1, FID2
Changed lines of the file:
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@@
   (wire (pts (xy 163.83 160.02) (xy 163.83 171.45)) (stroke (width 0) (type default)))
   (wire (pts (xy 163.83 171.45) (xy 168.91 171.45)) (stroke (width 0) (type default)))
-  (wire (pts (xy 129.54 162.56) (xy 135.89 162.56)) (stroke (width 0) (type default)))
-  (wire (pts (xy 129.54 135.89) (xy 129.54 162.56)) (stroke (width 0) (type default)))
+  (wire (pts (xy 134.62 162.56) (xy 135.89 162.56)) (stroke (width 0) (type default)))
+  (wire (pts (xy 134.62 135.89) (xy 134.62 162.56)) (stroke (width 0) (type default)))
+  (wire (pts (xy 74.93 135.89) (xy 129.54 135.89)) (stroke (width 0) (type default)))
+  (wire (pts (xy 129.54 135.89) (xy 134.62 135.89)) (stroke (width 0) (type default)))
   (wire (pts (xy 135.89 162.56) (xy 135.89 172.72)) (stroke (width 0) (type default)))
   (wire (pts (xy 135.89 172.72) (xy 168.91 172.72)) (stroke (width 0) (type default)))
@@
   (wire (pts (xy 69.85 134.62) (xy 74.93 134.62)) (stroke (width 0) (type default)))
   (wire (pts (xy 74.93 134.62) (xy 74.93 135.89)) (stroke (width 0) (type default)))
-  (wire (pts (xy 74.93 135.89) (xy 129.54 135.89)) (stroke (width 0) (type default)))
   (junction (at 39.37 100.33) (diameter 0) (color 0 0 0 0))
   (junction (at 69.85 100.33) (diameter 0) (color 0 0 0 0))
@@
     (instances (project "opamp-filter" (path "/efb028ab-a5b5-5d27-b654-08a8ba6b5d9d" (reference "H2") (unit 1))))
   )
-  (symbol (lib_id "Mechanical:Fiducial") (at 50.8 166.37 0.0) (unit 1)
-    (exclude_from_sim no) (in_bom no) (on_board yes) (dnp no)
-    (property "Reference" "FID1" (at 49.53 162.56 0) (effects (font (size 1.27 1.27)) (justify right)))
-    (property "Value" "Fiducial" (at 54.61 168.91 0) (effects (font (size 1.27 1.27)) (justify left) hide))
-    (property "Footprint" "Fiducial:Fiducial_1mm_Mask2mm" (at 50.8 166.37 0) (effects (font (size 1.27 1.27)) hide))
-    (property "Datasheet" "~" (at 50.8 166.37 0) (effects (font (size 1.27 1.27)) hide))
-    (property "MPN" "n/a" (at 50.8 166.37 0) (effects (font (size 1.27 1.27)) hide))
-    (property "Manufacturer" "n/a" (at 50.8 166.37 0) (effects (font (size 1.27 1.27)) hide))
+  (symbol (lib_id "Mechanical:MountingHole") (at 50.8 181.61 0.0) (unit 1)
+    (exclude_from_sim no) (in_bom no) (on_board yes) (dnp no)
+    (property "Reference" "H3" (at 49.53 177.8 0) (effects (font (size 1.27 1.27)) (justify right)))
+    (property "Value" "M3" (at 54.61 184.15 0) (effects (font (size 1.27 1.27)) (justify left) hide))
+    (property "Footprint" "MountingHole:MountingHole_3.2mm_M3" (at 50.8 181.61 0) (effects (font (size 1.27 1.27)) hide))
+    (property "Datasheet" "~" (at 50.8 181.61 0) (effects (font (size 1.27 1.27)) hide))
+    (property "MPN" "n/a" (at 50.8 181.61 0) (effects (font (size 1.27 1.27)) hide))
+    (property "Manufacturer" "n/a" (at 50.8 181.61 0) (effects (font (size 1.27 1.27)) hide))
+    (instances (project "opamp-filter" (path "/efb028ab-a5b5-5d27-b654-08a8ba6b5d9d" (reference "H3") (unit 1))))
+  )
+  (symbol (lib_id "Mechanical:Fiducial") (at 114.3 166.37 0.0) (unit 1)
+    (exclude_from_sim no) (in_bom no) (on_board yes) (dnp no)
+    (property "Reference" "FID1" (at 115.57 162.56 0) (effects (font (size 1.27 1.27)) (justify left)))
+    (property "Value" "Fiducial" (at 118.11 168.91 0) (effects (font (size 1.27 1.27)) (justify left) hide))
+    (property "Footprint" "Fiducial:Fiducial_1mm_Mask2mm" (at 114.3 166.37 0) (effects (font (size 1.27 1.27)) hide))
+    (property "Datasheet" "~" (at 114.3 166.37 0) (effects (font (size 1.27 1.27)) hide))
+    (property "MPN" "n/a" (at 114.3 166.37 0) (effects (font (size 1.27 1.27)) hide))
+    (property "Manufacturer" "n/a" (at 114.3 166.37 0) (effects (font (size 1.27 1.27)) hide))
     (instances (project "opamp-filter" (path "/efb028ab-a5b5-5d27-b654-08a8ba6b5d9d" (reference "FID1") (unit 1))))
   )
-  (symbol (lib_id "Mechanical:Fiducial") (at 63.5 166.37 0.0) (unit 1)
-    (exclude_from_sim no) (in_bom no) (on_board yes) (dnp no)
-    (property "Reference" "FID2" (at 62.23 162.56 0) (effects (font (size 1.27 1.27)) (justify right)))
-    (property "Value" "Fiducial" (at 54.61 168.91 0) (effects (font (size 1.27 1.27)) (justify right) hide))
-    (property "Footprint" "Fiducial:Fiducial_1mm_Mask2mm" (at 63.5 166.37 0) (effects (font (size 1.27 1.27)) hide))
-    (property "Datasheet" "~" (at 63.5 166.37 0) (effects (font (size 1.27 1.27)) hide))
-    (property "MPN" "n/a" (at 63.5 166.37 0) (effects (font (size 1.27 1.27)) hide))
-    (property "Manufacturer" "n/a" (at 63.5 166.37 0) (effects (font (size 1.27 1.27)) hide))
+  (symbol (lib_id "Mechanical:Fiducial") (at 127.0 166.37 0.0) (unit 1)
+    (exclude_from_sim no) (in_bom no) (on_board yes) (dnp no)
+    (property "Reference" "FID2" (at 127.0 162.56 0) (effects (font (size 1.27 1.27))))
+    (property "Value" "Fiducial" (at 118.11 168.91 0) (effects (font (size 1.27 1.27)) (justify right) hide))
+    (property "Footprint" "Fiducial:Fiducial_1mm_Mask2mm" (at 127.0 166.37 0) (effects (font (size 1.27 1.27)) hide))
+    (property "Datasheet" "~" (at 127.0 166.37 0) (effects (font (size 1.27 1.27)) hide))
+    (property "MPN" "n/a" (at 127.0 166.37 0) (effects (font (size 1.27 1.27)) hide))
+    (property "Manufacturer" "n/a" (at 127.0 166.37 0) (effects (font (size 1.27 1.27)) hide))
     (instances (project "opamp-filter" (path "/efb028ab-a5b5-5d27-b654-08a8ba6b5d9d" (reference "FID2") (unit 1))))
   )
