File: examples/pico-carrier/reviewed/pico-carrier.kicad_sch (KiCad schematic)
At the start: 9 parts, among them J1 5V IN, J3 GP0-GP15, J4 GP16-GP28, PWR, U1 Pico

Commit message: Read the five as an engineer would, and make the toolkit act on it
examples/REVIEW.md is the pass: the five designs read for circuit theory,
layout physics and readability, every finding dispatched to one of four
places - a rule, a fix, a reasoned waiver, or named as open. The headline
result: every reviewed/ project now PASSES its own gate, every as-generated/
still fails it, and every waiver is an engineering argument a reviewer can
disagree with.

Four new rules, each calibrated against KiCad's 18 human-drawn demo projects:

* readability.label_only - the sheet connects by name, not by wire; the
  single most recognisable mark of a generated schematic. 0 findings on the
  human corpus, 71-100% on ours.
* analog.no_dc_path - a net of only capacitors and connectors has nothing
  setting its DC level. Found a real fault: the op-amp filter's AC-coupled
  output floated. 0 findings on the corpus.
* route.detour - routed copper against the MST of the net's pads; the scenic
  tour an autorouter takes. 8 human boards fired at 2.5x, 0 at the shipped 4x.
* route.return_path - signal running over cuts in the other layer's ground
  fill, computed from the difference between a zone's outline and its fill,
  which the parser now keeps. Fires on 4 real demo boards, because real
  two-layer boards genuinely have the disease.

Three rules re-judged on evidence instead of names:

* analog.missing_decoupling reads pin electrical types: only power_in pins
  ask for a capacitor, and a net an output pin drives is never asked - a cap
  on an op-amp output is somebody's control loop. Retires the VBUS/VREF
  false positives without a single waiver.
* track.thin_power measures the longest contiguous narrow run against a
  power_neck_mm allowance. Pad entries and fine-pitch escapes pass; thin
  trunks still fail. 9 demo boards fired before, 0 after - all nine were necks.
* net.single_pin honours no-connect flags: a flagged pin is a decision.

And the designs themselves got the fixes the pa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
Changed lines of the file:
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@@
   (title_block
   	(title "Raspberry Pi Pico carrier, 5 V in")
-  	(date "2026-08-11")
+  	(date "2026-08-12")
   	(rev "A")
   	(company "kicad_skills examples")
-  	(comment 1 "generated 2026-08-11 by Claude Code (claude-opus-5)")
+  	(comment 1 "generated 2026-08-12 by Claude Code (claude-fable-5)")
   	(comment 2 "from tools/make_examples.py in sabas0ba/kicad_skills")
   )
+  (wire (pts (xy 119.38 110.49) (xy 72.39 110.49)) (stroke (width 0) (type default)))
+  (wire (pts (xy 119.38 113.03) (xy 72.39 113.03)) (stroke (width 0) (type default)))
+  (wire (pts (xy 119.38 115.57) (xy 72.39 115.57)) (stroke (width 0) (type default)))
+  (wire (pts (xy 119.38 118.11) (xy 72.39 118.11)) (stroke (width 0) (type default)))
   (wire (pts (xy 127.0 77.47) (xy 119.38 77.47)) (stroke (width 0) (type default)))
   (label "RUN" (at 119.38 77.47 0) (effects (font (size 1.27 1.27)) (justify left bottom)))
@@
   )
   (wire (pts (xy 64.77 110.49) (xy 72.39 110.49)) (stroke (width 0) (type default)))
-  (label "GP10" (at 72.39 110.49 0) (effects (font (size 1.27 1.27)) (justify left bottom)))
   (wire (pts (xy 64.77 113.03) (xy 72.39 113.03)) (stroke (width 0) (type default)))
-  (label "GP11" (at 72.39 113.03 0) (effects (font (size 1.27 1.27)) (justify left bottom)))
   (wire (pts (xy 64.77 115.57) (xy 72.39 115.57)) (stroke (width 0) (type default)))
-  (label "GP12" (at 72.39 115.57 0) (effects (font (size 1.27 1.27)) (justify left bottom)))
   (wire (pts (xy 64.77 118.11) (xy 72.39 118.11)) (stroke (width 0) (type default)))
-  (label "GP13" (at 72.39 118.11 0) (effects (font (size 1.27 1.27)) (justify left bottom)))
   (wire (pts (xy 64.77 120.65) (xy 72.39 120.65)) (stroke (width 0) (type default)))
   (symbol (lib_id "power:GND") (at 72.39 120.65 270) (unit 1)
