File: examples/fpga-audio/as-generated/fpga-audio.kicad_pcb (KiCad board)
At the start: 2 copper layers, 100 x 84 mm, 29 parts, among them J1 3V3 IN, J2 AUDIO OUT, J3 SPI PROG, U1 iCE40UP5K, U2 PCM5102A, U3 AP2112K-1.2, U4 W25Q32JV, X1 12MHz

Commit message: Keep the wire tree between runs too, and stop asking twice
Profiling what a regeneration actually costs turned up the real answer,
and it was not the router. The sheet's wire planner takes six minutes on
the FPGA example - it joins every signal net into a tree of straight, L
and Z runs that miss every other net's stub - and it was being asked for
the same answer twice per variant, by the shorts check and by the
emitter, neither of which knew the other had asked.

So it is memoised in the process and cached on disk beside the routing,
keyed by everything it reads: the parts and where they sit, the nets,
the notes, and its own source.

Two hot loops got a coarse grid index while the profile was open: the
sheet shorts check, which compared every wire against every other, and
the field placer, which asks "does this box touch any of those" a
hundred times per symbol against a thousand wires.

fpga-audio, both caches warm: 40 minutes to 17 seconds, and the four
smaller boards write byte-identical output.
Parts:
- moved C2 14.5 mm to (107.7, 80.8)
- moved C1 10.6 mm to (107.7, 77.3)
Routing:
- net /CRESET: track 177.0 -> 162.7 mm
- net /CLK12: track 31.2 -> 38.1 mm
- net +3V3: track 635.4 -> 629.1 mm
- net /+1V2: track 118.8 -> 115.1 mm
- net /OUTL: track 24.5 -> 27.2 mm
- net /SPI_SO: track 120.0 -> 122.3 mm
- net /OUTR: track 68.2 -> 66.0 mm
- net GND: track 135.3 -> 134.5 mm
- net /SPI_SS: track 85.6 -> 86.3 mm
