File: examples/fpga-audio/as-generated/fpga-audio.kicad_sch (KiCad schematic)
At the start: 29 parts, among them J1 3V3 IN, J2 AUDIO OUT, J3 SPI PROG, U1 iCE40UP5K, U2 PCM5102A, U3 AP2112K-1.2, U4 W25Q32JV, X1 12MHz

Commit message: Regenerate all five on the round-thirteen rules, and write the round down
The four fast boards pass their gates; measured across all five there are
zero crossings, zero doubled runs, zero mid-run width steps, every pour
piece over 8 mm2 holds its own via, and the shell reaches to 1.2 mm of
every edge. The FPGA sheet's two power blocks move clear of the frame -
the extended margin rule caught the second one this round. Its board
still fails, and the debt now has one name: four SPI nets at 11-20 mm
over plane cuts, two corners, and three detours all on the 3.3 V rail,
the twenty-link net that wants the same stated spine the 1.2 V rail got.
REVIEW.md section 18 records the round.

Co-Authored-By: Claude Fable 5 <noreply@anthropic.com>
Claude-Session: https://claude.ai/code/session_01DUj7Ltu92tWg159mCSacwY
Other:
- moved on the sheet: J1, J2
Changed lines of the file:
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@@
     (instances (project "fpga-audio" (path "/434dea94-d96f-5288-b60c-67317d440f4e" (reference "X1") (unit 1))))
   )
-  (wire (pts (xy 25.71 39.18) (xy 23.17 39.18)) (stroke (width 0) (type default)))
-  (wire (pts (xy 25.71 41.72) (xy 23.17 41.72)) (stroke (width 0) (type default)))
-  (symbol (lib_id "Connector:Screw_Terminal_01x02") (at 30.79 39.18 0.0) (unit 1)
-    (exclude_from_sim no) (in_bom yes) (on_board yes) (dnp no)
-    (property "Reference" "J1" (at 29.52 35.37 0) (effects (font (size 1.27 1.27)) (justify right)))
-    (property "Value" "3V3 IN" (at 34.6 44.26 0) (effects (font (size 1.27 1.27)) (justify left)))
-    (property "Footprint" "TerminalBlock_Phoenix:TerminalBlock_Phoenix_MKDS-1,5-2_1x02_P5.00mm_Horizontal" (at 30.79 39.18 0) (effects (font (size 1.27 1.27)) hide))
-    (property "Datasheet" "https://www.phoenixcontact.com/product/1729128" (at 30.79 39.18 0) (effects (font (size 1.27 1.27)) hide))
+  (wire (pts (xy 37.14 39.18) (xy 34.6 39.18)) (stroke (width 0) (type default)))
+  (wire (pts (xy 37.14 41.72) (xy 34.6 41.72)) (stroke (width 0) (type default)))
+  (symbol (lib_id "Connector:Screw_Terminal_01x02") (at 42.22 39.18 0.0) (unit 1)
+    (exclude_from_sim no) (in_bom yes) (on_board yes) (dnp no)
+    (property "Reference" "J1" (at 42.22 34.1 0) (effects (font (size 1.27 1.27))))
+    (property "Value" "3V3 IN" (at 35.87 44.26 0) (effects (font (size 1.27 1.27)) (justify right)))
+    (property "Footprint" "TerminalBlock_Phoenix:TerminalBlock_Phoenix_MKDS-1,5-2_1x02_P5.00mm_Horizontal" (at 42.22 39.18 0) (effects (font (size 1.27 1.27)) hide))
+    (property "Datasheet" "https://www.phoenixcontact.com/product/1729128" (at 42.22 39.18 0) (effects (font (size 1.27 1.27)) hide))
     (pin "1" (uuid "cad9b9e4-2eee-562a-a42a-31ca8c464aca-p1"))
     (pin "2" (uuid "cad9b9e4-2eee-562a-a42a-31ca8c464aca-p2"))
     (instances (project "fpga-audio" (path "/434dea94-d96f-5288-b60c-67317d440f4e" (reference "J1") (unit 1))))
   )
-  (wire (pts (xy 400.36 107.76) (xy 402.9 107.76)) (stroke (width 0) (type default)))
-  (label "OUTR" (at 402.9 107.76 0) (effects (font (size 1.27 1.27)) (justify left bottom)))
-  (wire (pts (xy 400.36 110.3) (xy 402.9 110.3)) (stroke (width 0) (type default)))
-  (wire (pts (xy 400.36 112.84) (xy 402.9 112.84)) (stroke (width 0) (type default)))
-  (label "OUTL" (at 402.9 112.84 0) (effects (font (size 1.27 1.27)) (justify left bottom)))
-  (symbol (lib_id "Connector:Conn_01x03_Pin") (at 395.28 110.3 0.0) (unit 1)
-    (exclude_from_sim no) (in_bom yes) (on_board yes) (dnp no)
-    (property "Reference" "J2" (at 394.01 106.363 0) (effects (font (size 1.27 1.27)) (justify right)))
-    (property "Value" "AUDIO OUT" (at 394.01 114.237 0) (effects (font (size 1.27 1.27)) (justify right)))
-    (property "Footprint" "Connector_PinHeader_2.54mm:PinHeader_1x03_P2.54mm_Vertical" (at 395.28 110.3 0) (effects (font (size 1.27 1.27)) hide))
-    (property "Datasheet" "https://www.we-online.com/components/products/datasheet/61300311121.pdf" (at 395.28 110.3 0) (effects (font (size 1.27 1.27)) hide))
+  (wire (pts (xy 394.01 107.76) (xy 396.55 107.76)) (stroke (width 0) (type default)))
+  (label "OUTR" (at 396.55 107.76 0) (effects (font (size 1.27 1.27)) (justify left bottom)))
+  (wire (pts (xy 394.01 110.3) (xy 396.55 110.3)) (stroke (width 0) (type default)))
+  (wire (pts (xy 394.01 112.84) (xy 396.55 112.84)) (stroke (width 0) (type default)))
+  (label "OUTL" (at 396.55 112.84 0) (effects (font (size 1.27 1.27)) (justify left bottom)))
+  (symbol (lib_id "Connector:Conn_01x03_Pin") (at 388.93 110.3 0.0) (unit 1)
+    (exclude_from_sim no) (in_bom yes) (on_board yes) (dnp no)
+    (property "Reference" "J2" (at 387.66 106.363 0) (effects (font (size 1.27 1.27)) (justify right)))
+    (property "Value" "AUDIO OUT" (at 387.66 114.237 0) (effects (font (size 1.27 1.27)) (justify right)))
+    (property "Footprint" "Connector_PinHeader_2.54mm:PinHeader_1x03_P2.54mm_Vertical" (at 388.93 110.3 0) (effects (font (size 1.27 1.27)) hide))
+    (property "Datasheet" "https://www.we-online.com/components/products/datasheet/61300311121.pdf" (at 388.93 110.3 0) (effects (font (size 1.27 1.27)) hide))
     (pin "1" (uuid "bcba810e-1eb1-5887-8060-8956a7b0e250-p1"))
     (pin "2" (uuid "bcba810e-1eb1-5887-8060-8956a7b0e250-p2"))
@@
   (wire (pts (xy 46.03 149.67) (xy 38.41 149.67)) (stroke (width 0) (type default)))
   (wire (pts (xy 38.41 136.97) (xy 38.41 149.67)) (stroke (width 0) (type default)))
-  (wire (pts (xy 23.17 39.18) (xy 15.55 39.18)) (stroke (width 0) (type default)))
-  (wire (pts (xy 15.55 34.1) (xy 15.55 39.18)) (stroke (width 0) (type default)))
-  (wire (pts (xy 23.17 41.72) (xy 13.01 41.72)) (stroke (width 0) (type default)))
-  (wire (pts (xy 13.01 41.72) (xy 13.01 49.34)) (stroke (width 0) (type default)))
-  (wire (pts (xy 402.9 110.3) (xy 410.52 110.3)) (stroke (width 0) (type default)))
-  (wire (pts (xy 410.52 110.3) (xy 410.52 117.92)) (stroke (width 0) (type default)))
+  (wire (pts (xy 34.6 39.18) (xy 26.98 39.18)) (stroke (width 0) (type default)))
+  (wire (pts (xy 26.98 34.1) (xy 26.98 39.18)) (stroke (width 0) (type default)))
+  (wire (pts (xy 34.6 41.72) (xy 24.44 41.72)) (stroke (width 0) (type default)))
+  (wire (pts (xy 24.44 41.72) (xy 24.44 49.34)) (stroke (width 0) (type default)))
+  (wire (pts (xy 396.55 110.3) (xy 404.17 110.3)) (stroke (width 0) (type default)))
+  (wire (pts (xy 404.17 110.3) (xy 404.17 117.92)) (stroke (width 0) (type default)))
   (wire (pts (xy 260.66 247.46) (xy 253.04 247.46)) (stroke (width 0) (type default)))
   (wire (pts (xy 253.04 247.46) (xy 253.04 252.54)) (stroke (width 0) (type default)))
@@
     (instances (project "fpga-audio" (path "/434dea94-d96f-5288-b60c-67317d440f4e" (reference "#PWR21") (unit 1))))
   )
-  (symbol (lib_id "power:+3V3") (at 15.55 34.1 0) (unit 1)
-    (exclude_from_sim no) (in_bom no) (on_board yes) (dnp no)
-    (property "Reference" "#PWR22" (at 15.55 34.1 0) (effects (font (size 1.27 1.27)) hide))
-    (property "Value" "+3V3" (at 15.55 30.29 0) (effects (font (size 1.27 1.27))))
-    (property "Footprint" "" (at 15.55 34.1 0) (effects (font (size 1.27 1.27)) hide))
-    (property "Datasheet" "" (at 15.55 34.1 0) (effects (font (size 1.27 1.27)) hide))
+  (symbol (lib_id "power:+3V3") (at 26.98 34.1 0) (unit 1)
+    (exclude_from_sim no) (in_bom no) (on_board yes) (dnp no)
+    (property "Reference" "#PWR22" (at 26.98 34.1 0) (effects (font (size 1.27 1.27)) hide))
+    (property "Value" "+3V3" (at 26.98 30.29 0) (effects (font (size 1.27 1.27))))
+    (property "Footprint" "" (at 26.98 34.1 0) (effects (font (size 1.27 1.27)) hide))
+    (property "Datasheet" "" (at 26.98 34.1 0) (effects (font (size 1.27 1.27)) hide))
     (pin "1" (uuid "050afbed-dbf0-5cec-900c-940c7a099fc7-p"))
     (instances (project "fpga-audio" (path "/434dea94-d96f-5288-b60c-67317d440f4e" (reference "#PWR22") (unit 1))))
   )
-  (symbol (lib_id "power:GND") (at 13.01 49.34 0) (unit 1)
-    (exclude_from_sim no) (in_bom no) (on_board yes) (dnp no)
-    (property "Reference" "#PWR23" (at 13.01 49.34 0) (effects (font (size 1.27 1.27)) hide))
-    (property "Value" "GND" (at 13.01 53.15 0) (effects (font (size 1.27 1.27))))
-    (property "Footprint" "" (at 13.01 49.34 0) (effects (font (size 1.27 1.27)) hide))
-    (property "Datasheet" "" (at 13.01 49.34 0) (effects (font (size 1.27 1.27)) hide))
+  (symbol (lib_id "power:GND") (at 24.44 49.34 0) (unit 1)
+    (exclude_from_sim no) (in_bom no) (on_board yes) (dnp no)
+    (property "Reference" "#PWR23" (at 24.44 49.34 0) (effects (font (size 1.27 1.27)) hide))
+    (property "Value" "GND" (at 24.44 53.15 0) (effects (font (size 1.27 1.27))))
+    (property "Footprint" "" (at 24.44 49.34 0) (effects (font (size 1.27 1.27)) hide))
+    (property "Datasheet" "" (at 24.44 49.34 0) (effects (font (size 1.27 1.27)) hide))
     (pin "1" (uuid "c7878787-c335-545c-b2a7-7952b8733c6c-p"))
     (instances (project "fpga-audio" (path "/434dea94-d96f-5288-b60c-67317d440f4e" (reference "#PWR23") (unit 1))))
   )
-  (symbol (lib_id "power:GND") (at 410.52 117.92 0) (unit 1)
-    (exclude_from_sim no) (in_bom no) (on_board yes) (dnp no)
-    (property "Reference" "#PWR24" (at 410.52 117.92 0) (effects (font (size 1.27 1.27)) hide))
-    (property "Value" "GND" (at 410.52 121.73 0) (effects (font (size 1.27 1.27))))
-    (property "Footprint" "" (at 410.52 117.92 0) (effects (font (size 1.27 1.27)) hide))
-    (property "Datasheet" "" (at 410.52 117.92 0) (effects (font (size 1.27 1.27)) hide))
+  (symbol (lib_id "power:GND") (at 404.17 117.92 0) (unit 1)
+    (exclude_from_sim no) (in_bom no) (on_board yes) (dnp no)
+    (property "Reference" "#PWR24" (at 404.17 117.92 0) (effects (font (size 1.27 1.27)) hide))
+    (property "Value" "GND" (at 404.17 121.73 0) (effects (font (size 1.27 1.27))))
+    (property "Footprint" "" (at 404.17 117.92 0) (effects (font (size 1.27 1.27)) hide))
+    (property "Datasheet" "" (at 404.17 117.92 0) (effects (font (size 1.27 1.27)) hide))
     (pin "1" (uuid "535b8bd9-6366-5d71-a2ff-37420f61cbf6-p"))
     (instances (project "fpga-audio" (path "/434dea94-d96f-5288-b60c-67317d440f4e" (reference "#PWR24") (unit 1))))

Commit message: Put the vias back where the copper moved, and let the fillets vote
The FPGA board came back from its re-route with two unconnected nets and
three dangling ends, and the cause was older than anything this round
added. The router hands back a via for every layer change; six passes
then reshape the copper - snapping to 45s, chamfering, spreading folds,
and now filleting - and none of them move the holes underneath. A joint
that slides a millimetre from its via is two loose ends and one broken
net, and `_unlooped` then swept the via away as orphaned, because it
kept a via only when a track ended on its exact coordinate.

Two fixes, both about what "connected" means. A via lives if kept copper
*touches* it, not if a coordinate matches. And a new `_joined` pass
re-derives the joints from the copper that actually got written: where a
net ends on two layers at one point with no via reaching it, one goes
back in. It reads the finished geometry, so it cannot drift the way six
separate passes carrying vias along with them would.

The same reasoning fixes two rules that had been measuring coordinates
rather than copper. `route.stub` matched a track end to a via's centre
exactly, and called a joint a stub whenever a reshaping pass had moved
it a quarter of a millimetre inside the very barrel it was connected to.
`route.width_step` walked a neck back to its pad and stopped at the
first width change - which, on a filleted board, is the teardrop, so
every escape's neck stopped being recognised as one.

While the three copies of the post-route pipeline were being edited for
the third time this session, they became one function. That is how
`_teardrops` had come to run on two of the three exits.

All five boards: DRC clean on both matrix versions, nothing unconnected.
Four pass their gates; the FPGA board is down to the two-layer bill it
has always had - four nets over plane cuts and one 88 degree corner.

Co-Authored-By: Claude Fable 5 <noreply@anthropic.com>
Claude-Session: https:/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
Parts:
- added FID1, FID2, FID3: Fiducial, Fiducial:Fiducial_1mm_Mask2mm, symbol Mechanical:Fiducial
- added H1, H2, H3, H4: M3, MountingHole:MountingHole_3.2mm_M3, symbol Mechanical:MountingHole
Connections:
- net +3V3: no longer C15.1, C3.1, C4.1, R3.1, U1.30 (VCC), U1.5 (VCC), U3.5 (VOUT)
- net GND: no longer R2.2, U1.7 (CDONE)
- new net +1V2: C15.1, C3.1, C4.1, R3.1, U1.30 (VCC), U1.5 (VCC), U3.5 (VOUT)
- new net CDONE: R2.2, U1.7 (CDONE)
Other:
- moved on the sheet: C15
Changed lines of the file:
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@@
     (instances (project "fpga-audio" (path "/434dea94-d96f-5288-b60c-67317d440f4e" (reference "R2") (unit 1))))
   )
-  (wire (pts (xy 140.01 228.41) (xy 140.01 225.87)) (stroke (width 0) (type default)))
-  (label "+1V2" (at 140.01 225.87 90) (effects (font (size 1.27 1.27)) (justify left bottom)))
-  (wire (pts (xy 140.01 236.03) (xy 140.01 238.57)) (stroke (width 0) (type default)))
-  (symbol (lib_id "Device:C") (at 140.01 232.22 0.0) (unit 1)
+  (wire (pts (xy 148.9 58.23) (xy 148.9 55.69)) (stroke (width 0) (type default)))
+  (label "+1V2" (at 148.9 55.69 90) (effects (font (size 1.27 1.27)) (justify left bottom)))
+  (wire (pts (xy 148.9 65.85) (xy 148.9 68.39)) (stroke (width 0) (type default)))
+  (symbol (lib_id "Device:C") (at 148.9 62.04 0.0) (unit 1)
     (exclude_from_sim no) (in_bom yes) (on_board yes) (dnp no)
-    (property "Reference" "C15" (at 137.47 227.14 0) (effects (font (size 1.27 1.27)) (justify right)))
-    (property "Value" "100n" (at 136.2 237.3 0) (effects (font (size 1.27 1.27)) (justify right)))
-    (property "Footprint" "Capacitor_SMD:C_0603_1608Metric" (at 140.01 232.22 0) (effects (font (size 1.27 1.27)) hide))
-    (property "Datasheet" "https://product.samsungsem.com/mlcc/CL10B104KB8NNNC.do" (at 140.01 232.22 0) (effects (font (size 1.27 1.27)) hide))
+    (property "Reference" "C15" (at 147.63 55.69 0) (effects (font (size 1.27 1.27)) (justify right)))
+    (property "Value" "100n" (at 152.71 67.12 0) (effects (font (size 1.27 1.27)) (justify left)))
+    (property "Footprint" "Capacitor_SMD:C_0603_1608Metric" (at 148.9 62.04 0) (effects (font (size 1.27 1.27)) hide))
+    (property "Datasheet" "https://product.samsungsem.com/mlcc/CL10B104KB8NNNC.do" (at 148.9 62.04 0) (effects (font (size 1.27 1.27)) hide))
     (pin "1" (uuid "b43e868f-badc-5d7e-89b5-2f3614e8bb24-p1"))
     (pin "2" (uuid "b43e868f-badc-5d7e-89b5-2f3614e8bb24-p2"))
     (instances (project "fpga-audio" (path "/434dea94-d96f-5288-b60c-67317d440f4e" (reference "C15") (unit 1))))
+  )
+  (symbol (lib_id "Mechanical:MountingHole") (at 292.41 237.3 0.0) (unit 1)
+    (exclude_from_sim no) (in_bom no) (on_board yes) (dnp no)
+    (property "Reference" "H1" (at 291.14 233.49 0) (effects (font (size 1.27 1.27)) (justify right)))
+    (property "Value" "M3" (at 296.22 239.84 0) (effects (font (size 1.27 1.27)) (justify left) hide))
+    (property "Footprint" "MountingHole:MountingHole_3.2mm_M3" (at 292.41 237.3 0) (effects (font (size 1.27 1.27)) hide))
+    (property "Datasheet" "~" (at 292.41 237.3 0) (effects (font (size 1.27 1.27)) hide))
+    (instances (project "fpga-audio" (path "/434dea94-d96f-5288-b60c-67317d440f4e" (reference "H1") (unit 1))))
+  )
+  (symbol (lib_id "Mechanical:MountingHole") (at 305.11 237.3 0.0) (unit 1)
+    (exclude_from_sim no) (in_bom no) (on_board yes) (dnp no)
+    (property "Reference" "H2" (at 303.84 233.49 0) (effects (font (size 1.27 1.27)) (justify right)))
+    (property "Value" "M3" (at 308.92 239.84 0) (effects (font (size 1.27 1.27)) (justify left) hide))
+    (property "Footprint" "MountingHole:MountingHole_3.2mm_M3" (at 305.11 237.3 0) (effects (font (size 1.27 1.27)) hide))
+    (property "Datasheet" "~" (at 305.11 237.3 0) (effects (font (size 1.27 1.27)) hide))
+    (instances (project "fpga-audio" (path "/434dea94-d96f-5288-b60c-67317d440f4e" (reference "H2") (unit 1))))
+  )
+  (symbol (lib_id "Mechanical:MountingHole") (at 317.81 237.3 0.0) (unit 1)
+    (exclude_from_sim no) (in_bom no) (on_board yes) (dnp no)
+    (property "Reference" "H3" (at 316.54 233.49 0) (effects (font (size 1.27 1.27)) (justify right)))
+    (property "Value" "M3" (at 321.62 239.84 0) (effects (font (size 1.27 1.27)) (justify left) hide))
+    (property "Footprint" "MountingHole:MountingHole_3.2mm_M3" (at 317.81 237.3 0) (effects (font (size 1.27 1.27)) hide))
+    (property "Datasheet" "~" (at 317.81 237.3 0) (effects (font (size 1.27 1.27)) hide))
+    (instances (project "fpga-audio" (path "/434dea94-d96f-5288-b60c-67317d440f4e" (reference "H3") (unit 1))))
+  )
+  (symbol (lib_id "Mechanical:MountingHole") (at 330.51 237.3 0.0) (unit 1)
+    (exclude_from_sim no) (in_bom no) (on_board yes) (dnp no)
+    (property "Reference" "H4" (at 329.24 233.49 0) (effects (font (size 1.27 1.27)) (justify right)))
+    (property "Value" "M3" (at 334.32 239.84 0) (effects (font (size 1.27 1.27)) (justify left) hide))
+    (property "Footprint" "MountingHole:MountingHole_3.2mm_M3" (at 330.51 237.3 0) (effects (font (size 1.27 1.27)) hide))
+    (property "Datasheet" "~" (at 330.51 237.3 0) (effects (font (size 1.27 1.27)) hide))
+    (instances (project "fpga-audio" (path "/434dea94-d96f-5288-b60c-67317d440f4e" (reference "H4") (unit 1))))
+  )
+  (symbol (lib_id "Mechanical:Fiducial") (at 216.21 222.06 0.0) (unit 1)
+    (exclude_from_sim no) (in_bom no) (on_board yes) (dnp no)
+    (property "Reference" "FID1" (at 214.94 218.25 0) (effects (font (size 1.27 1.27)) (justify right)))
+    (property "Value" "Fiducial" (at 220.02 224.6 0) (effects (font (size 1.27 1.27)) (justify left) hide))
+    (property "Footprint" "Fiducial:Fiducial_1mm_Mask2mm" (at 216.21 222.06 0) (effects (font (size 1.27 1.27)) hide))
+    (property "Datasheet" "~" (at 216.21 222.06 0) (effects (font (size 1.27 1.27)) hide))
+    (instances (project "fpga-audio" (path "/434dea94-d96f-5288-b60c-67317d440f4e" (reference "FID1") (unit 1))))
+  )
+  (symbol (lib_id "Mechanical:Fiducial") (at 228.91 222.06 0.0) (unit 1)
+    (exclude_from_sim no) (in_bom no) (on_board yes) (dnp no)
+    (property "Reference" "FID2" (at 227.64 218.25 0) (effects (font (size 1.27 1.27)) (justify right)))
+    (property "Value" "Fiducial" (at 232.72 224.6 0) (effects (font (size 1.27 1.27)) (justify left) hide))
+    (property "Footprint" "Fiducial:Fiducial_1mm_Mask2mm" (at 228.91 222.06 0) (effects (font (size 1.27 1.27)) hide))
+    (property "Datasheet" "~" (at 228.91 222.06 0) (effects (font (size 1.27 1.27)) hide))
+    (instances (project "fpga-audio" (path "/434dea94-d96f-5288-b60c-67317d440f4e" (reference "FID2") (unit 1))))
+  )
+  (symbol (lib_id "Mechanical:Fiducial") (at 228.91 222.06 0.0) (unit 1)
+    (exclude_from_sim no) (in_bom no) (on_board yes) (dnp no)
+    (property "Reference" "FID3" (at 230.18 218.25 0) (effects (font (size 1.27 1.27)) (justify left)))
+    (property "Value" "Fiducial" (at 220.02 224.6 0) (effects (font (size 1.27 1.27)) (justify right) hide))
+    (property "Footprint" "Fiducial:Fiducial_1mm_Mask2mm" (at 228.91 222.06 0) (effects (font (size 1.27 1.27)) hide))
+    (property "Datasheet" "~" (at 228.91 222.06 0) (effects (font (size 1.27 1.27)) hide))
+    (instances (project "fpga-audio" (path "/434dea94-d96f-5288-b60c-67317d440f4e" (reference "FID3") (unit 1))))
   )
   (wire (pts (xy 311.46 117.92) (xy 303.84 117.92)) (stroke (width 0) (type default)))
@@
     (exclude_from_sim no) (in_bom no) (on_board yes) (dnp no)
     (property "Reference" "#PWR52" (at 140.01 225.87 0) (effects (font (size 1.27 1.27)) hide))
-    (property "Value" "+3V3" (at 142.55 222.06 0) (effects (font (size 1.27 1.27)) (justify left)))
+    (property "Value" "+3V3" (at 140.01 222.06 0) (effects (font (size 1.27 1.27))))
     (property "Footprint" "" (at 140.01 225.87 0) (effects (font (size 1.27 1.27)) hide))
     (property "Datasheet" "" (at 140.01 225.87 0) (effects (font (size 1.27 1.27)) hide))
@@
     (instances (project "fpga-audio" (path "/434dea94-d96f-5288-b60c-67317d440f4e" (reference "#PWR52") (unit 1))))
   )
-  (symbol (lib_id "power:GND") (at 140.01 238.57 0) (unit 1)
-    (exclude_from_sim no) (in_bom no) (on_board yes) (dnp no)
-    (property "Reference" "#PWR53" (at 140.01 238.57 0) (effects (font (size 1.27 1.27)) hide))
-    (property "Value" "GND" (at 142.55 242.38 0) (effects (font (size 1.27 1.27)) (justify left)))
-    (property "Footprint" "" (at 140.01 238.57 0) (effects (font (size 1.27 1.27)) hide))
-    (property "Datasheet" "" (at 140.01 238.57 0) (effects (font (size 1.27 1.27)) hide))
+  (symbol (lib_id "power:GND") (at 148.9 68.39 0) (unit 1)
+    (exclude_from_sim no) (in_bom no) (on_board yes) (dnp no)
+    (property "Reference" "#PWR53" (at 148.9 68.39 0) (effects (font (size 1.27 1.27)) hide))
+    (property "Value" "GND" (at 148.9 72.2 0) (effects (font (size 1.27 1.27))))
+    (property "Footprint" "" (at 148.9 68.39 0) (effects (font (size 1.27 1.27)) hide))
+    (property "Datasheet" "" (at 148.9 68.39 0) (effects (font (size 1.27 1.27)) hide))
     (pin "1" (uuid "a2262622-9b7f-5bc7-9be1-32de81b27a83-p"))
     (instances (project "fpga-audio" (path "/434dea94-d96f-5288-b60c-67317d440f4e" (reference "#PWR53") (unit 1))))
