File: examples/fpga-audio/as-generated/fpga-audio.kicad_sch (KiCad schematic)
At the start: 36 parts, among them J1 3V3 IN, J2 AUDIO OUT, J3 SPI PROG, U1 iCE40UP5K, U2 PCM5102A, U3 AP2112K-1.2, U4 W25Q32JV, X1 12MHz

Commit message: Rebuild golden layouts and gate floorplan quality
Connections:
- net CRESET: now also J3.3 (Pin_3); no longer J3.5 (Pin_5)
- net GND: now also J2.3 (Pin_3); no longer J2.2 (Pin_2)
- net OUTL: now also J2.2 (Pin_2); no longer J2.3 (Pin_3)
- net SPI_SCK: now also J3.4 (Pin_4); no longer J3.2 (Pin_2)
- net SPI_SI: now also J3.5 (Pin_5); no longer J3.3 (Pin_3)
- net SPI_SO: now also J3.2 (Pin_2); no longer J3.4 (Pin_4)
Changed lines of the file:
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@@
   (paper "A3")
   (title_block
-  	(comment 1 "generated 2026-08-12 by Claude Code (claude-fable-5)")
-  	(comment 2 "from tools/make_examples.py in sabas0ba/kicad_skills")
+    (comment 1 "generated 2026-09-05 by OpenAI Codex")
+    (comment 2 "from tools/make_examples.py in sabas0ba/kicad_skills")
   )
   (no_connect (at 185.73 95.06))
@@
   (label "OUTR" (at 396.55 107.76 0) (effects (font (size 1.27 1.27)) (justify left bottom)))
   (wire (pts (xy 394.01 110.3) (xy 396.55 110.3)) (stroke (width 0) (type default)))
+  (label "OUTL" (at 396.55 110.3 0) (effects (font (size 1.27 1.27)) (justify left bottom)))
   (wire (pts (xy 394.01 112.84) (xy 396.55 112.84)) (stroke (width 0) (type default)))
-  (label "OUTL" (at 396.55 112.84 0) (effects (font (size 1.27 1.27)) (justify left bottom)))
   (symbol (lib_id "Connector:Conn_01x03_Pin") (at 388.93 110.3 0.0) (unit 1)
     (exclude_from_sim no) (in_bom yes) (on_board yes) (dnp no)
@@
   (label "SPI_SS" (at 260.66 234.76 0) (effects (font (size 1.27 1.27)) (justify right bottom)))
   (wire (pts (xy 263.2 237.3) (xy 260.66 237.3)) (stroke (width 0) (type default)))
-  (label "SPI_SCK" (at 260.66 237.3 0) (effects (font (size 1.27 1.27)) (justify right bottom)))
+  (label "SPI_SO" (at 260.66 237.3 0) (effects (font (size 1.27 1.27)) (justify right bottom)))
   (wire (pts (xy 263.2 239.84) (xy 260.66 239.84)) (stroke (width 0) (type default)))
-  (label "SPI_SI" (at 260.66 239.84 0) (effects (font (size 1.27 1.27)) (justify right bottom)))
+  (label "CRESET" (at 260.66 239.84 0) (effects (font (size 1.27 1.27)) (justify right bottom)))
   (wire (pts (xy 263.2 242.38) (xy 260.66 242.38)) (stroke (width 0) (type default)))
-  (label "SPI_SO" (at 260.66 242.38 0) (effects (font (size 1.27 1.27)) (justify right bottom)))
+  (label "SPI_SCK" (at 260.66 242.38 0) (effects (font (size 1.27 1.27)) (justify right bottom)))
   (wire (pts (xy 263.2 244.92) (xy 260.66 244.92)) (stroke (width 0) (type default)))
-  (label "CRESET" (at 260.66 244.92 0) (effects (font (size 1.27 1.27)) (justify right bottom)))
+  (label "SPI_SI" (at 260.66 244.92 0) (effects (font (size 1.27 1.27)) (justify right bottom)))
   (wire (pts (xy 263.2 247.46) (xy 260.66 247.46)) (stroke (width 0) (type default)))
   (symbol (lib_id "Connector:Conn_01x06_Pin") (at 268.28 239.84 0.0) (mirror y) (unit 1)
@@
   (wire (pts (xy 34.6 41.72) (xy 24.44 41.72)) (stroke (width 0) (type default)))
   (wire (pts (xy 24.44 41.72) (xy 24.44 49.34)) (stroke (width 0) (type default)))
-  (wire (pts (xy 396.55 110.3) (xy 404.17 110.3)) (stroke (width 0) (type default)))
-  (wire (pts (xy 404.17 110.3) (xy 404.17 117.92)) (stroke (width 0) (type default)))
+  (wire (pts (xy 396.55 112.84) (xy 404.17 112.84)) (stroke (width 0) (type default)))
+  (wire (pts (xy 404.17 112.84) (xy 404.17 117.92)) (stroke (width 0) (type default)))
   (wire (pts (xy 260.66 247.46) (xy 253.04 247.46)) (stroke (width 0) (type default)))
   (wire (pts (xy 253.04 247.46) (xy 253.04 252.54)) (stroke (width 0) (type default)))
