File: examples/fpga-audio/as-generated/fpga-audio.kicad_sch (KiCad schematic)
At the start: 35 parts, among them J1 3V3 IN, J2 AUDIO OUT, J3 SPI PROG, U1 iCE40UP5K, U2 PCM5102A, U3 AP2112K-1.2, U4 W25Q32JV, X1 12MHz

Commit message: Move the corner that belongs to neither track
route.acute_angle reads copper, not the objects the copper was written from,
so it sees two corners no pass could: a joint where a run of one width meets a
run of another, and a pair of segments eighteen microns long left by a chamfer
of a chamfer - an 88 degree corner on a run that is visibly straight.

_welded takes both. The debris comes out where a point has debris on each side,
so a genuinely short leg into a pad keeps its shape. The joint moves: the two
far ends stay put and the point between them becomes the elbow that joins them
without reversing, each track keeping one leg and its own width.

_pinned_points is deliberately not what holds a joint still - that set pins
every track end, because moving one of a pair leaves the other in mid air,
which is the case this pass exists for and handles by moving both. What may
not move is a pad or a via.

fpga-audio is down to two: three nets over cuts in the plane, and one run that
tours. The other four stay at 0 errors, 0 warnings.

Co-Authored-By: Claude Fable 5 <noreply@anthropic.com>
Claude-Session: https://claude.ai/code/session_01DUj7Ltu92tWg159mCSacwY
Parts:
- added FID3: Fiducial, Fiducial:Fiducial_1mm_Mask2mm, symbol Mechanical:Fiducial
Other:
- moved on the sheet: FID2
Changed lines of the file:
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@@
     (instances (project "fpga-audio" (path "/434dea94-d96f-5288-b60c-67317d440f4e" (reference "FID1") (unit 1))))
   )
-  (symbol (lib_id "Mechanical:Fiducial") (at 216.21 222.06 0.0) (unit 1)
+  (symbol (lib_id "Mechanical:Fiducial") (at 228.91 222.06 0.0) (unit 1)
     (exclude_from_sim no) (in_bom no) (on_board yes) (dnp no)
-    (property "Reference" "FID2" (at 217.48 218.25 0) (effects (font (size 1.27 1.27)) (justify left)))
-    (property "Value" "Fiducial" (at 212.4 224.6 0) (effects (font (size 1.27 1.27)) (justify right) hide))
-    (property "Footprint" "Fiducial:Fiducial_1mm_Mask2mm" (at 216.21 222.06 0) (effects (font (size 1.27 1.27)) hide))
-    (property "Datasheet" "~" (at 216.21 222.06 0) (effects (font (size 1.27 1.27)) hide))
+    (property "Reference" "FID2" (at 227.64 218.25 0) (effects (font (size 1.27 1.27)) (justify right)))
+    (property "Value" "Fiducial" (at 232.72 224.6 0) (effects (font (size 1.27 1.27)) (justify left) hide))
+    (property "Footprint" "Fiducial:Fiducial_1mm_Mask2mm" (at 228.91 222.06 0) (effects (font (size 1.27 1.27)) hide))
+    (property "Datasheet" "~" (at 228.91 222.06 0) (effects (font (size 1.27 1.27)) hide))
     (instances (project "fpga-audio" (path "/434dea94-d96f-5288-b60c-67317d440f4e" (reference "FID2") (unit 1))))
   )
+  (symbol (lib_id "Mechanical:Fiducial") (at 228.91 222.06 0.0) (unit 1)
+    (exclude_from_sim no) (in_bom no) (on_board yes) (dnp no)
+    (property "Reference" "FID3" (at 230.18 218.25 0) (effects (font (size 1.27 1.27)) (justify left)))
+    (property "Value" "Fiducial" (at 220.02 224.6 0) (effects (font (size 1.27 1.27)) (justify right) hide))
+    (property "Footprint" "Fiducial:Fiducial_1mm_Mask2mm" (at 228.91 222.06 0) (effects (font (size 1.27 1.27)) hide))
+    (property "Datasheet" "~" (at 228.91 222.06 0) (effects (font (size 1.27 1.27)) hide))
+    (instances (project "fpga-audio" (path "/434dea94-d96f-5288-b60c-67317d440f4e" (reference "FID3") (unit 1))))
+  )
   (wire (pts (xy 311.46 117.92) (xy 303.84 117.92)) (stroke (width 0) (type default)))

Commit message: feat(examples): round twenty - fuse and clamp every input, state the ESR, damp the clock, control the mute
Redesign of the five worked examples for the items REVIEW.md left open:

- every power input gets a fuse in series and a TVS across the fused rail
  (a resettable fuse on the Pico carrier, whose Schottky already blocks a
  reversed supply); each sheet states what the clamp does not do
- the buck's output capacitor states the ESR the LM2596 loop is designed
  around (SNVS124G 9.1.3), derived from the ripple already on the sheet
- the FPGA's 12 MHz clock leaves its oscillator through 33 ohms
- the DAC's XSMT is driven from the FPGA with a pull-down instead of
  strapped high, so it comes up muted
- the op-amp filter's output goes through a 100 ohm isolation resistor

Generator fixes the round found: _surfaced pruned a via that tapped the
middle of a back-layer spine, and _chamfer_tracks cut the copper out from
under a via sitting a fraction along a leg; both left a net in two pieces
that KiCad's DRC reported. Pin stubs closer than 7.62 mm draw over each
other, so the new parts are spaced for it and the comments say why.

tools/example_images.py renders the README pictures from the regenerated
projects. All five reviewed variants pass their gates and KiCad's DRC on
both matrix versions; the as-generated variants each carry one more
blocking finding (spec.missing_esr). REVIEW.md 25 records the round.

Co-Authored-By: Claude Fable 5.1 <noreply@anthropic.com>
Claude-Session: https://claude.ai/code/session_017JKofiLFxXjzRRnBmFyXuQ
Parts:
- added D3: SMAJ5.0A, Diode_SMD:D_SMA, symbol Device:D_Zener
- added F1: 500mA, Fuse:Fuse_1206_3216Metric, symbol Device:Fuse
- added R5: 33R, Resistor_SMD:R_0603_1608Metric, symbol Device:R
- added R6: 10k, Resistor_SMD:R_0603_1608Metric, symbol Device:R
Connections:
- net +3V3: now also D3.1 (K), F1.2; no longer J1.1 (Pin_1), U2.17 (XSMT)
- net CLK12: now also R5.2; no longer X1.3 (OUT)
- net GND: now also D3.2 (A), R6.2
- net XSMT: now reaches U1.31 (IOT_42b)
- net XSMT: now also U2.17 (XSMT), R6.1
- new net OSC_OUT: R5.1, X1.3 (OUT)
- new net VIN: F1.1, J1.1 (Pin_1)
- no-connect marks 31 -> 30
Other:
- moved on the sheet: C3, C4, C9, J1, U3
