File: examples/motor-driver/as-generated/motor-driver.kicad_sch (KiCad schematic)
At the start: 17 parts, among them J1 VM 2.7-10.8V, J2 MOTOR A, J3 MOTOR B, J4 LOGIC, U1 DRV8833PW

Commit message: Walk the whole edge for a screw hole, and land a joint on its own pad
The fastener clearance was right and the search was not: it slid along two
edges from each corner and gave up, so boards that had had four screw holes
came back with one. It now walks a ring round the board at the inset the
screw needs, taking the nearest free point to each corner - and only from
that corner's own quarter, because a search that asked for the nearest free
point anywhere put three of the four along one edge, each of them the nearest
thing to a different corner. A quarter with no room gives no screw: three
that hold the board flat beat four that hold one side.

A pin header asks for nothing above its courtyard - the socket that fits it
lands inside the outline the header already draws - while a screw terminal's
wires leave horizontally from its face. Treating the two alike is what left a
carrier lined with headers with two holes on one edge. Both the generator and
the rule now tell them apart by footprint.

_landed folds a via that sits beside a plated hole of its own net onto the
hole. The plating already joins the faces, so the via bought nothing and cost
hole-to-hole: two drills a millimetre apart leave 0.15 mm of laminate at a
0.25 mm rule, which is what DRC reported on the opamp board.

The fillets move to the end of the pipeline. A taper is built against the end
of a run, and _landed moves ends, so a teardrop laid before it pointed at
where the run used to stop - a nought-degree corner in the angle rule.

buck-5v, motor-driver, pico-carrier, opamp-filter: 0 errors, 0 warnings.

Co-Authored-By: Claude Fable 5 <noreply@anthropic.com>
Claude-Session: https://claude.ai/code/session_01DUj7Ltu92tWg159mCSacwY
Parts:
- added FID3: Fiducial, Fiducial:Fiducial_1mm_Mask2mm, symbol Mechanical:Fiducial
- added H4: M3, MountingHole:MountingHole_3.2mm_M3_Pad, symbol Mechanical:MountingHole_Pad
Connections:
- net GND: now also H4.1
Other:
- moved on the sheet: FID1, FID2
Changed lines of the file:
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@@
     (instances (project "motor-driver" (path "/bddeec65-fa67-5f6a-9af2-d98e98d56e38" (reference "H3") (unit 1))))
   )
-  (symbol (lib_id "Mechanical:Fiducial") (at 63.81 149.67 0.0) (unit 1)
+  (wire (pts (xy 63.81 152.21) (xy 63.81 154.75)) (stroke (width 0) (type default)))
+  (symbol (lib_id "Mechanical:MountingHole_Pad") (at 63.81 149.67 0.0) (unit 1)
     (exclude_from_sim no) (in_bom no) (on_board yes) (dnp no)
-    (property "Reference" "FID1" (at 62.54 145.86 0) (effects (font (size 1.27 1.27)) (justify right)))
-    (property "Value" "Fiducial" (at 67.62 152.21 0) (effects (font (size 1.27 1.27)) (justify left) hide))
-    (property "Footprint" "Fiducial:Fiducial_1mm_Mask2mm" (at 63.81 149.67 0) (effects (font (size 1.27 1.27)) hide))
+    (property "Reference" "H4" (at 62.54 144.59 0) (effects (font (size 1.27 1.27)) (justify right)))
+    (property "Value" "M3" (at 67.62 153.48 0) (effects (font (size 1.27 1.27)) (justify left) hide))
+    (property "Footprint" "MountingHole:MountingHole_3.2mm_M3_Pad" (at 63.81 149.67 0) (effects (font (size 1.27 1.27)) hide))
     (property "Datasheet" "~" (at 63.81 149.67 0) (effects (font (size 1.27 1.27)) hide))
+    (pin "1" (uuid "742cc603-3332-588e-9d01-92620b38e2a8-p1"))
+    (instances (project "motor-driver" (path "/bddeec65-fa67-5f6a-9af2-d98e98d56e38" (reference "H4") (unit 1))))
+  )
+  (symbol (lib_id "Mechanical:Fiducial") (at 76.51 149.67 0.0) (unit 1)
+    (exclude_from_sim no) (in_bom no) (on_board yes) (dnp no)
+    (property "Reference" "FID1" (at 75.24 145.86 0) (effects (font (size 1.27 1.27)) (justify right)))
+    (property "Value" "Fiducial" (at 80.32 152.21 0) (effects (font (size 1.27 1.27)) (justify left) hide))
+    (property "Footprint" "Fiducial:Fiducial_1mm_Mask2mm" (at 76.51 149.67 0) (effects (font (size 1.27 1.27)) hide))
+    (property "Datasheet" "~" (at 76.51 149.67 0) (effects (font (size 1.27 1.27)) hide))
     (instances (project "motor-driver" (path "/bddeec65-fa67-5f6a-9af2-d98e98d56e38" (reference "FID1") (unit 1))))
   )
-  (symbol (lib_id "Mechanical:Fiducial") (at 63.81 149.67 0.0) (unit 1)
+  (symbol (lib_id "Mechanical:Fiducial") (at 89.21 149.67 0.0) (unit 1)
     (exclude_from_sim no) (in_bom no) (on_board yes) (dnp no)
-    (property "Reference" "FID2" (at 65.08 145.86 0) (effects (font (size 1.27 1.27)) (justify left)))
-    (property "Value" "Fiducial" (at 65.08 154.75 0) (effects (font (size 1.27 1.27)) (justify left) hide))
-    (property "Footprint" "Fiducial:Fiducial_1mm_Mask2mm" (at 63.81 149.67 0) (effects (font (size 1.27 1.27)) hide))
-    (property "Datasheet" "~" (at 63.81 149.67 0) (effects (font (size 1.27 1.27)) hide))
+    (property "Reference" "FID2" (at 87.94 145.86 0) (effects (font (size 1.27 1.27)) (justify right)))
+    (property "Value" "Fiducial" (at 93.02 152.21 0) (effects (font (size 1.27 1.27)) (justify left) hide))
+    (property "Footprint" "Fiducial:Fiducial_1mm_Mask2mm" (at 89.21 149.67 0) (effects (font (size 1.27 1.27)) hide))
+    (property "Datasheet" "~" (at 89.21 149.67 0) (effects (font (size 1.27 1.27)) hide))
     (instances (project "motor-driver" (path "/bddeec65-fa67-5f6a-9af2-d98e98d56e38" (reference "FID2") (unit 1))))
+  )
+  (symbol (lib_id "Mechanical:Fiducial") (at 89.21 149.67 0.0) (unit 1)
+    (exclude_from_sim no) (in_bom no) (on_board yes) (dnp no)
+    (property "Reference" "FID3" (at 90.48 145.86 0) (effects (font (size 1.27 1.27)) (justify left)))
+    (property "Value" "Fiducial" (at 90.48 154.75 0) (effects (font (size 1.27 1.27)) (justify left) hide))
+    (property "Footprint" "Fiducial:Fiducial_1mm_Mask2mm" (at 89.21 149.67 0) (effects (font (size 1.27 1.27)) hide))
+    (property "Datasheet" "~" (at 89.21 149.67 0) (effects (font (size 1.27 1.27)) hide))
+    (instances (project "motor-driver" (path "/bddeec65-fa67-5f6a-9af2-d98e98d56e38" (reference "FID3") (unit 1))))
   )
   (wire (pts (xy 46.03 82.36) (xy 53.65 82.36)) (stroke (width 0) (type default)))
@@
     (instances (project "motor-driver" (path "/bddeec65-fa67-5f6a-9af2-d98e98d56e38" (reference "#PWR11") (unit 1))))
   )
+  (symbol (lib_id "power:GND") (at 63.81 154.75 0) (unit 1)
+    (exclude_from_sim no) (in_bom no) (on_board yes) (dnp no)
+    (property "Reference" "#PWR12" (at 63.81 154.75 0) (effects (font (size 1.27 1.27)) hide))
+    (property "Value" "GND" (at 63.81 158.56 0) (effects (font (size 1.27 1.27))))
+    (property "Footprint" "" (at 63.81 154.75 0) (effects (font (size 1.27 1.27)) hide))
+    (property "Datasheet" "" (at 63.81 154.75 0) (effects (font (size 1.27 1.27)) hide))
+    (pin "1" (uuid "3b9627af-8076-5306-88c7-4bd3286e9f17-p"))
+    (instances (project "motor-driver" (path "/bddeec65-fa67-5f6a-9af2-d98e98d56e38" (reference "#PWR12") (unit 1))))
+  )
   (junction (at 106.99 77.28) (diameter 0) (color 0 0 0 0))
