File: examples/motor-driver/as-generated/motor-driver.kicad_sch (KiCad schematic)
At the start: 19 parts, among them J1 VM 2.7-10.8V, J2 MOTOR A, J3 MOTOR B, J4 LOGIC, U1 DRV8833PW

Commit message: Rebuild golden layouts and gate floorplan quality
Parts:
- removed H4: M3, MountingHole:MountingHole_3.2mm_M3_Pad, symbol Mechanical:MountingHole_Pad
Other:
- moved on the sheet: FID1, FID2, FID3
Changed lines of the file:
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@@
   (paper "A4")
   (title_block
-  	(comment 1 "generated 2026-08-12 by Claude Code (claude-fable-5)")
-  	(comment 2 "from tools/make_examples.py in sabas0ba/kicad_skills")
+    (comment 1 "generated 2026-09-05 by OpenAI Codex")
+    (comment 2 "from tools/make_examples.py in sabas0ba/kicad_skills")
   )
   (wire (pts (xy 43.49 79.82) (xy 46.03 79.82)) (stroke (width 0) (type default)))
@@
     (instances (project "motor-driver" (path "/bddeec65-fa67-5f6a-9af2-d98e98d56e38" (reference "H3") (unit 1))))
   )
-  (wire (pts (xy 63.81 152.21) (xy 63.81 154.75)) (stroke (width 0) (type default)))
-  (symbol (lib_id "Mechanical:MountingHole_Pad") (at 63.81 149.67 0.0) (unit 1)
-    (exclude_from_sim no) (in_bom no) (on_board yes) (dnp no)
-    (property "Reference" "H4" (at 62.54 144.59 0) (effects (font (size 1.27 1.27)) (justify right)))
-    (property "Value" "M3" (at 67.62 153.48 0) (effects (font (size 1.27 1.27)) (justify left) hide))
-    (property "Footprint" "MountingHole:MountingHole_3.2mm_M3_Pad" (at 63.81 149.67 0) (effects (font (size 1.27 1.27)) hide))
+  (symbol (lib_id "Mechanical:Fiducial") (at 63.81 149.67 0.0) (unit 1)
+    (exclude_from_sim no) (in_bom no) (on_board yes) (dnp no)
+    (property "Reference" "FID1" (at 62.54 145.86 0) (effects (font (size 1.27 1.27)) (justify right)))
+    (property "Value" "Fiducial" (at 67.62 152.21 0) (effects (font (size 1.27 1.27)) (justify left) hide))
+    (property "Footprint" "Fiducial:Fiducial_1mm_Mask2mm" (at 63.81 149.67 0) (effects (font (size 1.27 1.27)) hide))
     (property "Datasheet" "~" (at 63.81 149.67 0) (effects (font (size 1.27 1.27)) hide))
-    (pin "1" (uuid "742cc603-3332-588e-9d01-92620b38e2a8-p1"))
-    (instances (project "motor-driver" (path "/bddeec65-fa67-5f6a-9af2-d98e98d56e38" (reference "H4") (unit 1))))
+    (instances (project "motor-driver" (path "/bddeec65-fa67-5f6a-9af2-d98e98d56e38" (reference "FID1") (unit 1))))
   )
   (symbol (lib_id "Mechanical:Fiducial") (at 76.51 149.67 0.0) (unit 1)
     (exclude_from_sim no) (in_bom no) (on_board yes) (dnp no)
-    (property "Reference" "FID1" (at 75.24 145.86 0) (effects (font (size 1.27 1.27)) (justify right)))
+    (property "Reference" "FID2" (at 75.24 145.86 0) (effects (font (size 1.27 1.27)) (justify right)))
     (property "Value" "Fiducial" (at 80.32 152.21 0) (effects (font (size 1.27 1.27)) (justify left) hide))
     (property "Footprint" "Fiducial:Fiducial_1mm_Mask2mm" (at 76.51 149.67 0) (effects (font (size 1.27 1.27)) hide))
     (property "Datasheet" "~" (at 76.51 149.67 0) (effects (font (size 1.27 1.27)) hide))
-    (instances (project "motor-driver" (path "/bddeec65-fa67-5f6a-9af2-d98e98d56e38" (reference "FID1") (unit 1))))
-  )
-  (symbol (lib_id "Mechanical:Fiducial") (at 89.21 149.67 0.0) (unit 1)
-    (exclude_from_sim no) (in_bom no) (on_board yes) (dnp no)
-    (property "Reference" "FID2" (at 87.94 145.86 0) (effects (font (size 1.27 1.27)) (justify right)))
-    (property "Value" "Fiducial" (at 93.02 152.21 0) (effects (font (size 1.27 1.27)) (justify left) hide))
-    (property "Footprint" "Fiducial:Fiducial_1mm_Mask2mm" (at 89.21 149.67 0) (effects (font (size 1.27 1.27)) hide))
-    (property "Datasheet" "~" (at 89.21 149.67 0) (effects (font (size 1.27 1.27)) hide))
     (instances (project "motor-driver" (path "/bddeec65-fa67-5f6a-9af2-d98e98d56e38" (reference "FID2") (unit 1))))
   )
-  (symbol (lib_id "Mechanical:Fiducial") (at 89.21 149.67 0.0) (unit 1)
-    (exclude_from_sim no) (in_bom no) (on_board yes) (dnp no)
-    (property "Reference" "FID3" (at 90.48 145.86 0) (effects (font (size 1.27 1.27)) (justify left)))
-    (property "Value" "Fiducial" (at 90.48 154.75 0) (effects (font (size 1.27 1.27)) (justify left) hide))
-    (property "Footprint" "Fiducial:Fiducial_1mm_Mask2mm" (at 89.21 149.67 0) (effects (font (size 1.27 1.27)) hide))
-    (property "Datasheet" "~" (at 89.21 149.67 0) (effects (font (size 1.27 1.27)) hide))
+  (symbol (lib_id "Mechanical:Fiducial") (at 76.51 149.67 0.0) (unit 1)
+    (exclude_from_sim no) (in_bom no) (on_board yes) (dnp no)
+    (property "Reference" "FID3" (at 77.78 145.86 0) (effects (font (size 1.27 1.27)) (justify left)))
+    (property "Value" "Fiducial" (at 77.78 154.75 0) (effects (font (size 1.27 1.27)) (justify left) hide))
+    (property "Footprint" "Fiducial:Fiducial_1mm_Mask2mm" (at 76.51 149.67 0) (effects (font (size 1.27 1.27)) hide))
+    (property "Datasheet" "~" (at 76.51 149.67 0) (effects (font (size 1.27 1.27)) hide))
     (instances (project "motor-driver" (path "/bddeec65-fa67-5f6a-9af2-d98e98d56e38" (reference "FID3") (unit 1))))
   )
@@
     (instances (project "motor-driver" (path "/bddeec65-fa67-5f6a-9af2-d98e98d56e38" (reference "#PWR11") (unit 1))))
   )
-  (symbol (lib_id "power:GND") (at 63.81 154.75 0) (unit 1)
-    (exclude_from_sim no) (in_bom no) (on_board yes) (dnp no)
-    (property "Reference" "#PWR12" (at 63.81 154.75 0) (effects (font (size 1.27 1.27)) hide))
-    (property "Value" "GND" (at 63.81 158.56 0) (effects (font (size 1.27 1.27))))
-    (property "Footprint" "" (at 63.81 154.75 0) (effects (font (size 1.27 1.27)) hide))
-    (property "Datasheet" "" (at 63.81 154.75 0) (effects (font (size 1.27 1.27)) hide))
-    (pin "1" (uuid "3b9627af-8076-5306-88c7-4bd3286e9f17-p"))
-    (instances (project "motor-driver" (path "/bddeec65-fa67-5f6a-9af2-d98e98d56e38" (reference "#PWR12") (unit 1))))
-  )
   (junction (at 106.99 77.28) (diameter 0) (color 0 0 0 0))
