File: examples/motor-driver/as-generated/motor-driver.kicad_pcb (KiCad board)
At the start: 2 copper layers, 68 x 46 mm, 18 parts, among them J1 VM 2.7-10.8V, J2 MOTOR A, J3 MOTOR B, J4 LOGIC, U1 DRV8833PW

Commit message: Clear final motor layout blockers
Parts:
- moved D2 2.00 mm to (145.2, 65.8)
Routing:
- net /LED_A: track 11.6 -> 2.15 mm, vias 1 -> 0
- net GND: track 51.6 -> 56.7 mm, vias 0 -> 1
- net /AIN2: track 35.4 -> 39.2 mm, vias 2 -> 1
