File: examples/opamp-filter/as-generated/opamp-filter.kicad_sch (KiCad schematic)
At the start: 28 parts, among them J1 IN, J2 5V, J3 OUT, U1 MCP6001R, U2 MCP6001R

Commit message: Leave room for the screw, and print the ink where the board is
The screw holes were placed against the hole's own courtyard, which is the
drill plus a whisker - so on four of the five boards a hole sat inside a
connector's mating space, closest 0.42 mm. What goes through an M3 hole is a
pan head on a washer, seven millimetres of steel lying flat, and a connector
wants its shell, its wires and the fingers that fit them on top of that. The
spot search now keeps the fastener's own circle clear of every part body and
gives connectors CONNECTOR_ACCESS more, and three rules say so when a board
does not: mechanical.fastener_clearance, mechanical.connector_access and
mechanical.fastener_copper, all blocking for a generated design.

Silk was measured with a per-character advance of 0.78, and KiCad's stroke
font is proportional at 0.94 to 1.07. Everything downstream of that estimate
was placing ink where it did not fit: a legend across a capacitor's land, a
designator through the board's own name. `_text_extent` takes the top of the
measured range, adds the fab's clearance and is used by every silk placement.

Three placements also fell through to a position nobody chose. A designator
that found nothing kept its library offset, which for a part in a corner
points off the board; the board id took the first of eight fixed strips; a
legend took the least bad of six spots. All three are scored now, over
candidate sets wide enough to have an answer - and a pad-less footprint, which
is what a mounting hole is, is no longer skipped outright.

silk.off_board reports the case KiCad's own test cannot: ink that clears the
edge entirely is never printed, and DRC only measures ink that crosses it.

_unspiked redraws a corner tighter than a right angle as the elbow between its
neighbours - one diagonal, one straight, no step back to a heading the line
has already left. It is never longer than what it replaces.

All four fast boards: 0 errors, 0 warnings.

Co-Authored-By: Claude Fable 5 <no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
Parts:
- removed FID3: Fiducial, Fiducial:Fiducial_1mm_Mask2mm, symbol Mechanical:Fiducial
- removed H3: M3, MountingHole:MountingHole_3.2mm_M3, symbol Mechanical:MountingHole
Other:
- moved on the sheet: FID1, FID2, H1, H2
Changed lines of the file:
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@@
     (instances (project "opamp-filter" (path "/efb028ab-a5b5-5d27-b654-08a8ba6b5d9d" (reference "TP3") (unit 1))))
   )
-  (symbol (lib_id "Mechanical:MountingHole") (at 241.61 149.67 0.0) (unit 1)
+  (symbol (lib_id "Mechanical:MountingHole") (at 114.61 149.67 0.0) (unit 1)
     (exclude_from_sim no) (in_bom no) (on_board yes) (dnp no)
-    (property "Reference" "H1" (at 240.34 145.86 0) (effects (font (size 1.27 1.27)) (justify right)))
-    (property "Value" "M3" (at 245.42 152.21 0) (effects (font (size 1.27 1.27)) (justify left) hide))
-    (property "Footprint" "MountingHole:MountingHole_3.2mm_M3" (at 241.61 149.67 0) (effects (font (size 1.27 1.27)) hide))
-    (property "Datasheet" "~" (at 241.61 149.67 0) (effects (font (size 1.27 1.27)) hide))
+    (property "Reference" "H1" (at 113.34 145.86 0) (effects (font (size 1.27 1.27)) (justify right)))
+    (property "Value" "M3" (at 118.42 152.21 0) (effects (font (size 1.27 1.27)) (justify left) hide))
+    (property "Footprint" "MountingHole:MountingHole_3.2mm_M3" (at 114.61 149.67 0) (effects (font (size 1.27 1.27)) hide))
+    (property "Datasheet" "~" (at 114.61 149.67 0) (effects (font (size 1.27 1.27)) hide))
     (instances (project "opamp-filter" (path "/efb028ab-a5b5-5d27-b654-08a8ba6b5d9d" (reference "H1") (unit 1))))
   )
-  (symbol (lib_id "Mechanical:MountingHole") (at 254.31 149.67 0.0) (unit 1)
+  (symbol (lib_id "Mechanical:MountingHole") (at 127.31 149.67 0.0) (unit 1)
     (exclude_from_sim no) (in_bom no) (on_board yes) (dnp no)
-    (property "Reference" "H2" (at 253.04 145.86 0) (effects (font (size 1.27 1.27)) (justify right)))
-    (property "Value" "M3" (at 258.12 152.21 0) (effects (font (size 1.27 1.27)) (justify left) hide))
-    (property "Footprint" "MountingHole:MountingHole_3.2mm_M3" (at 254.31 149.67 0) (effects (font (size 1.27 1.27)) hide))
-    (property "Datasheet" "~" (at 254.31 149.67 0) (effects (font (size 1.27 1.27)) hide))
+    (property "Reference" "H2" (at 126.04 145.86 0) (effects (font (size 1.27 1.27)) (justify right)))
+    (property "Value" "M3" (at 131.12 152.21 0) (effects (font (size 1.27 1.27)) (justify left) hide))
+    (property "Footprint" "MountingHole:MountingHole_3.2mm_M3" (at 127.31 149.67 0) (effects (font (size 1.27 1.27)) hide))
+    (property "Datasheet" "~" (at 127.31 149.67 0) (effects (font (size 1.27 1.27)) hide))
     (instances (project "opamp-filter" (path "/efb028ab-a5b5-5d27-b654-08a8ba6b5d9d" (reference "H2") (unit 1))))
   )
-  (symbol (lib_id "Mechanical:MountingHole") (at 267.01 149.67 0.0) (unit 1)
+  (symbol (lib_id "Mechanical:Fiducial") (at 190.81 149.67 0.0) (unit 1)
     (exclude_from_sim no) (in_bom no) (on_board yes) (dnp no)
-    (property "Reference" "H3" (at 265.74 145.86 0) (effects (font (size 1.27 1.27)) (justify right)))
-    (property "Value" "M3" (at 270.82 152.21 0) (effects (font (size 1.27 1.27)) (justify left) hide))
-    (property "Footprint" "MountingHole:MountingHole_3.2mm_M3" (at 267.01 149.67 0) (effects (font (size 1.27 1.27)) hide))
-    (property "Datasheet" "~" (at 267.01 149.67 0) (effects (font (size 1.27 1.27)) hide))
-    (instances (project "opamp-filter" (path "/efb028ab-a5b5-5d27-b654-08a8ba6b5d9d" (reference "H3") (unit 1))))
-  )
-  (symbol (lib_id "Mechanical:Fiducial") (at 89.21 134.43 0.0) (unit 1)
-    (exclude_from_sim no) (in_bom no) (on_board yes) (dnp no)
-    (property "Reference" "FID1" (at 87.94 130.62 0) (effects (font (size 1.27 1.27)) (justify right)))
-    (property "Value" "Fiducial" (at 93.02 136.97 0) (effects (font (size 1.27 1.27)) (justify left) hide))
-    (property "Footprint" "Fiducial:Fiducial_1mm_Mask2mm" (at 89.21 134.43 0) (effects (font (size 1.27 1.27)) hide))
-    (property "Datasheet" "~" (at 89.21 134.43 0) (effects (font (size 1.27 1.27)) hide))
+    (property "Reference" "FID1" (at 190.81 145.86 0) (effects (font (size 1.27 1.27))))
+    (property "Value" "Fiducial" (at 194.62 152.21 0) (effects (font (size 1.27 1.27)) (justify left) hide))
+    (property "Footprint" "Fiducial:Fiducial_1mm_Mask2mm" (at 190.81 149.67 0) (effects (font (size 1.27 1.27)) hide))
+    (property "Datasheet" "~" (at 190.81 149.67 0) (effects (font (size 1.27 1.27)) hide))
     (instances (project "opamp-filter" (path "/efb028ab-a5b5-5d27-b654-08a8ba6b5d9d" (reference "FID1") (unit 1))))
   )
-  (symbol (lib_id "Mechanical:Fiducial") (at 101.91 134.43 0.0) (unit 1)
+  (symbol (lib_id "Mechanical:Fiducial") (at 190.81 149.67 0.0) (unit 1)
     (exclude_from_sim no) (in_bom no) (on_board yes) (dnp no)
-    (property "Reference" "FID2" (at 100.64 130.62 0) (effects (font (size 1.27 1.27)) (justify right)))
-    (property "Value" "Fiducial" (at 105.72 136.97 0) (effects (font (size 1.27 1.27)) (justify left) hide))
-    (property "Footprint" "Fiducial:Fiducial_1mm_Mask2mm" (at 101.91 134.43 0) (effects (font (size 1.27 1.27)) hide))
-    (property "Datasheet" "~" (at 101.91 134.43 0) (effects (font (size 1.27 1.27)) hide))
+    (property "Reference" "FID2" (at 194.62 147.13 0) (effects (font (size 1.27 1.27)) (justify left)))
+    (property "Value" "Fiducial" (at 179.38 152.21 0) (effects (font (size 1.27 1.27)) (justify right) hide))
+    (property "Footprint" "Fiducial:Fiducial_1mm_Mask2mm" (at 190.81 149.67 0) (effects (font (size 1.27 1.27)) hide))
+    (property "Datasheet" "~" (at 190.81 149.67 0) (effects (font (size 1.27 1.27)) hide))
     (instances (project "opamp-filter" (path "/efb028ab-a5b5-5d27-b654-08a8ba6b5d9d" (reference "FID2") (unit 1))))
   )
-  (symbol (lib_id "Mechanical:Fiducial") (at 101.91 134.43 0.0) (unit 1)
-    (exclude_from_sim no) (in_bom no) (on_board yes) (dnp no)
-    (property "Reference" "FID3" (at 103.18 130.62 0) (effects (font (size 1.27 1.27)) (justify left)))
-    (property "Value" "Fiducial" (at 93.02 136.97 0) (effects (font (size 1.27 1.27)) (justify right) hide))
-    (property "Footprint" "Fiducial:Fiducial_1mm_Mask2mm" (at 101.91 134.43 0) (effects (font (size 1.27 1.27)) hide))
-    (property "Datasheet" "~" (at 101.91 134.43 0) (effects (font (size 1.27 1.27)) hide))
-    (instances (project "opamp-filter" (path "/efb028ab-a5b5-5d27-b654-08a8ba6b5d9d" (reference "FID3") (unit 1))))
-  )
   (wire (pts (xy 38.41 102.68) (xy 46.03 102.68)) (stroke (width 0) (type default)))

Commit message: Walk the whole edge for a screw hole, and land a joint on its own pad
The fastener clearance was right and the search was not: it slid along two
edges from each corner and gave up, so boards that had had four screw holes
came back with one. It now walks a ring round the board at the inset the
screw needs, taking the nearest free point to each corner - and only from
that corner's own quarter, because a search that asked for the nearest free
point anywhere put three of the four along one edge, each of them the nearest
thing to a different corner. A quarter with no room gives no screw: three
that hold the board flat beat four that hold one side.

A pin header asks for nothing above its courtyard - the socket that fits it
lands inside the outline the header already draws - while a screw terminal's
wires leave horizontally from its face. Treating the two alike is what left a
carrier lined with headers with two holes on one edge. Both the generator and
the rule now tell them apart by footprint.

_landed folds a via that sits beside a plated hole of its own net onto the
hole. The plating already joins the faces, so the via bought nothing and cost
hole-to-hole: two drills a millimetre apart leave 0.15 mm of laminate at a
0.25 mm rule, which is what DRC reported on the opamp board.

The fillets move to the end of the pipeline. A taper is built against the end
of a run, and _landed moves ends, so a teardrop laid before it pointed at
where the run used to stop - a nought-degree corner in the angle rule.

buck-5v, motor-driver, pico-carrier, opamp-filter: 0 errors, 0 warnings.

Co-Authored-By: Claude Fable 5 <noreply@anthropic.com>
Claude-Session: https://claude.ai/code/session_01DUj7Ltu92tWg159mCSacwY
Parts:
- added FID3: Fiducial, Fiducial:Fiducial_1mm_Mask2mm, symbol Mechanical:Fiducial
Other:
- moved on the sheet: FID1, FID2
Changed lines of the file:
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@@
     (instances (project "opamp-filter" (path "/efb028ab-a5b5-5d27-b654-08a8ba6b5d9d" (reference "H2") (unit 1))))
   )
-  (symbol (lib_id "Mechanical:Fiducial") (at 190.81 149.67 0.0) (unit 1)
+  (symbol (lib_id "Mechanical:Fiducial") (at 241.61 149.67 0.0) (unit 1)
     (exclude_from_sim no) (in_bom no) (on_board yes) (dnp no)
-    (property "Reference" "FID1" (at 190.81 145.86 0) (effects (font (size 1.27 1.27))))
-    (property "Value" "Fiducial" (at 194.62 152.21 0) (effects (font (size 1.27 1.27)) (justify left) hide))
-    (property "Footprint" "Fiducial:Fiducial_1mm_Mask2mm" (at 190.81 149.67 0) (effects (font (size 1.27 1.27)) hide))
-    (property "Datasheet" "~" (at 190.81 149.67 0) (effects (font (size 1.27 1.27)) hide))
+    (property "Reference" "FID1" (at 240.34 145.86 0) (effects (font (size 1.27 1.27)) (justify right)))
+    (property "Value" "Fiducial" (at 245.42 152.21 0) (effects (font (size 1.27 1.27)) (justify left) hide))
+    (property "Footprint" "Fiducial:Fiducial_1mm_Mask2mm" (at 241.61 149.67 0) (effects (font (size 1.27 1.27)) hide))
+    (property "Datasheet" "~" (at 241.61 149.67 0) (effects (font (size 1.27 1.27)) hide))
     (instances (project "opamp-filter" (path "/efb028ab-a5b5-5d27-b654-08a8ba6b5d9d" (reference "FID1") (unit 1))))
   )
-  (symbol (lib_id "Mechanical:Fiducial") (at 190.81 149.67 0.0) (unit 1)
+  (symbol (lib_id "Mechanical:Fiducial") (at 254.31 149.67 0.0) (unit 1)
     (exclude_from_sim no) (in_bom no) (on_board yes) (dnp no)
-    (property "Reference" "FID2" (at 194.62 147.13 0) (effects (font (size 1.27 1.27)) (justify left)))
-    (property "Value" "Fiducial" (at 179.38 152.21 0) (effects (font (size 1.27 1.27)) (justify right) hide))
-    (property "Footprint" "Fiducial:Fiducial_1mm_Mask2mm" (at 190.81 149.67 0) (effects (font (size 1.27 1.27)) hide))
-    (property "Datasheet" "~" (at 190.81 149.67 0) (effects (font (size 1.27 1.27)) hide))
+    (property "Reference" "FID2" (at 253.04 145.86 0) (effects (font (size 1.27 1.27)) (justify right)))
+    (property "Value" "Fiducial" (at 258.12 152.21 0) (effects (font (size 1.27 1.27)) (justify left) hide))
+    (property "Footprint" "Fiducial:Fiducial_1mm_Mask2mm" (at 254.31 149.67 0) (effects (font (size 1.27 1.27)) hide))
+    (property "Datasheet" "~" (at 254.31 149.67 0) (effects (font (size 1.27 1.27)) hide))
     (instances (project "opamp-filter" (path "/efb028ab-a5b5-5d27-b654-08a8ba6b5d9d" (reference "FID2") (unit 1))))
   )
+  (symbol (lib_id "Mechanical:Fiducial") (at 254.31 149.67 0.0) (unit 1)
+    (exclude_from_sim no) (in_bom no) (on_board yes) (dnp no)
+    (property "Reference" "FID3" (at 255.58 145.86 0) (effects (font (size 1.27 1.27)) (justify left)))
+    (property "Value" "Fiducial" (at 245.42 152.21 0) (effects (font (size 1.27 1.27)) (justify right) hide))
+    (property "Footprint" "Fiducial:Fiducial_1mm_Mask2mm" (at 254.31 149.67 0) (effects (font (size 1.27 1.27)) hide))
+    (property "Datasheet" "~" (at 254.31 149.67 0) (effects (font (size 1.27 1.27)) hide))
+    (instances (project "opamp-filter" (path "/efb028ab-a5b5-5d27-b654-08a8ba6b5d9d" (reference "FID3") (unit 1))))
+  )
   (wire (pts (xy 38.41 102.68) (xy 46.03 102.68)) (stroke (width 0) (type default)))
