File: examples/buck-5v/as-generated/buck-5v.kicad_sch (KiCad schematic)
At the start: 17 parts, among them J1 12V IN, J2 5V OUT, U1 LM2596S-5

Commit message: Rebuild golden layouts and gate floorplan quality
Parts:
- removed H3: M3, MountingHole:MountingHole_3.2mm_M3, symbol Mechanical:MountingHole
Other:
- moved on the sheet: FID1, FID2, FID3
Changed lines of the file:
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@@
   (paper "A4")
   (title_block
-  	(comment 1 "generated 2026-08-12 by Claude Code (claude-fable-5)")
-  	(comment 2 "from tools/make_examples.py in sabas0ba/kicad_skills")
+    (comment 1 "generated 2026-09-05 by OpenAI Codex")
+    (comment 2 "from tools/make_examples.py in sabas0ba/kicad_skills")
   )
   (wire (pts (xy 43.49 63.31) (xy 46.03 63.31)) (stroke (width 0) (type default)))
@@
     (instances (project "buck-5v" (path "/ec98644d-848c-5056-a4cb-c829189be5c3" (reference "H2") (unit 1))))
   )
-  (symbol (lib_id "Mechanical:MountingHole") (at 51.11 149.67 0.0) (unit 1)
+  (symbol (lib_id "Mechanical:Fiducial") (at 51.11 149.67 0.0) (unit 1)
     (exclude_from_sim no) (in_bom no) (on_board yes) (dnp no)
-    (property "Reference" "H3" (at 49.84 145.86 0) (effects (font (size 1.27 1.27)) (justify right)))
-    (property "Value" "M3" (at 54.92 152.21 0) (effects (font (size 1.27 1.27)) (justify left) hide))
-    (property "Footprint" "MountingHole:MountingHole_3.2mm_M3" (at 51.11 149.67 0) (effects (font (size 1.27 1.27)) hide))
+    (property "Reference" "FID1" (at 49.84 145.86 0) (effects (font (size 1.27 1.27)) (justify right)))
+    (property "Value" "Fiducial" (at 54.92 152.21 0) (effects (font (size 1.27 1.27)) (justify left) hide))
+    (property "Footprint" "Fiducial:Fiducial_1mm_Mask2mm" (at 51.11 149.67 0) (effects (font (size 1.27 1.27)) hide))
     (property "Datasheet" "~" (at 51.11 149.67 0) (effects (font (size 1.27 1.27)) hide))
-    (instances (project "buck-5v" (path "/ec98644d-848c-5056-a4cb-c829189be5c3" (reference "H3") (unit 1))))
+    (instances (project "buck-5v" (path "/ec98644d-848c-5056-a4cb-c829189be5c3" (reference "FID1") (unit 1))))
   )
   (symbol (lib_id "Mechanical:Fiducial") (at 63.81 149.67 0.0) (unit 1)
     (exclude_from_sim no) (in_bom no) (on_board yes) (dnp no)
-    (property "Reference" "FID1" (at 62.54 145.86 0) (effects (font (size 1.27 1.27)) (justify right)))
+    (property "Reference" "FID2" (at 62.54 145.86 0) (effects (font (size 1.27 1.27)) (justify right)))
     (property "Value" "Fiducial" (at 67.62 152.21 0) (effects (font (size 1.27 1.27)) (justify left) hide))
     (property "Footprint" "Fiducial:Fiducial_1mm_Mask2mm" (at 63.81 149.67 0) (effects (font (size 1.27 1.27)) hide))
     (property "Datasheet" "~" (at 63.81 149.67 0) (effects (font (size 1.27 1.27)) hide))
-    (instances (project "buck-5v" (path "/ec98644d-848c-5056-a4cb-c829189be5c3" (reference "FID1") (unit 1))))
-  )
-  (symbol (lib_id "Mechanical:Fiducial") (at 76.51 149.67 0.0) (unit 1)
-    (exclude_from_sim no) (in_bom no) (on_board yes) (dnp no)
-    (property "Reference" "FID2" (at 75.24 145.86 0) (effects (font (size 1.27 1.27)) (justify right)))
-    (property "Value" "Fiducial" (at 80.32 152.21 0) (effects (font (size 1.27 1.27)) (justify left) hide))
-    (property "Footprint" "Fiducial:Fiducial_1mm_Mask2mm" (at 76.51 149.67 0) (effects (font (size 1.27 1.27)) hide))
-    (property "Datasheet" "~" (at 76.51 149.67 0) (effects (font (size 1.27 1.27)) hide))
     (instances (project "buck-5v" (path "/ec98644d-848c-5056-a4cb-c829189be5c3" (reference "FID2") (unit 1))))
   )
-  (symbol (lib_id "Mechanical:Fiducial") (at 76.51 149.67 0.0) (unit 1)
+  (symbol (lib_id "Mechanical:Fiducial") (at 63.81 149.67 0.0) (unit 1)
     (exclude_from_sim no) (in_bom no) (on_board yes) (dnp no)
-    (property "Reference" "FID3" (at 77.78 145.86 0) (effects (font (size 1.27 1.27)) (justify left)))
-    (property "Value" "Fiducial" (at 77.78 154.75 0) (effects (font (size 1.27 1.27)) (justify left) hide))
-    (property "Footprint" "Fiducial:Fiducial_1mm_Mask2mm" (at 76.51 149.67 0) (effects (font (size 1.27 1.27)) hide))
-    (property "Datasheet" "~" (at 76.51 149.67 0) (effects (font (size 1.27 1.27)) hide))
+    (property "Reference" "FID3" (at 65.08 145.86 0) (effects (font (size 1.27 1.27)) (justify left)))
+    (property "Value" "Fiducial" (at 65.08 154.75 0) (effects (font (size 1.27 1.27)) (justify left) hide))
+    (property "Footprint" "Fiducial:Fiducial_1mm_Mask2mm" (at 63.81 149.67 0) (effects (font (size 1.27 1.27)) hide))
+    (property "Datasheet" "~" (at 63.81 149.67 0) (effects (font (size 1.27 1.27)) hide))
     (instances (project "buck-5v" (path "/ec98644d-848c-5056-a4cb-c829189be5c3" (reference "FID3") (unit 1))))
   )
