File: examples/buck-5v/as-generated/buck-5v.kicad_sch (KiCad schematic)
At the start: 16 parts, among them J1 12V IN, J2 5V OUT, U1 LM2596S-5

Commit message: chore(examples): regenerate the four two-layer boards and their pictures
buck-5v, motor-driver, pico-carrier and opamp-filter, regenerated from the
merged generator and gated clean on KiCad 9.0.9. The inner-layer pictures go
with the inner layers.

fpga-audio is still routing; it follows.

Co-Authored-By: Claude Opus 5 <noreply@anthropic.com>
Claude-Session: https://claude.ai/code/session_01XQE7UkE9WTSMW3oZ3kLeCt
Parts:
- added D3: SMAJ18A, Diode_SMD:D_SMA, symbol Device:D_Zener
- added F1: 3A, Fuse:Fuse_1206_3216Metric, symbol Device:Fuse
Connections:
- net +12V: now also D3.1 (K), F1.2; no longer J1.1 (Pin_1)
- net GND: now also D3.2 (A)
- new net VIN: F1.1, J1.1 (Pin_1)
Other:
- moved on the sheet: C1, J1
