File: examples/buck-5v/reviewed/buck-5v.kicad_sch (KiCad schematic)
At the start: 17 parts, among them J1 12V IN, J2 5V OUT, U1 LM2596S-5

Commit message: Rebuild golden layouts and gate floorplan quality
Parts:
- removed H3: M3, MountingHole:MountingHole_3.2mm_M3, symbol Mechanical:MountingHole
Other:
- moved on the sheet: FID1, FID2, FID3
Changed lines of the file:
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@@
   (paper "A4")
   (title_block
-  	(title "12 V to 5 V buck converter, 2 A")
-  	(date "2026-08-12")
-  	(rev "A")
-  	(company "kicad_skills examples")
-  	(comment 1 "generated 2026-08-12 by Claude Code (claude-fable-5)")
-  	(comment 2 "from tools/make_examples.py in sabas0ba/kicad_skills")
+    (title "12 V to 5 V buck converter, 2 A")
+    (date "2026-09-05")
+    (rev "A")
+    (company "kicad_skills examples")
+    (comment 1 "generated 2026-09-05 by OpenAI Codex")
+    (comment 2 "from tools/make_examples.py in sabas0ba/kicad_skills")
   )
   (wire (pts (xy 215.9 100.33) (xy 215.9 101.6)) (stroke (width 0) (type default)))
@@
     (instances (project "buck-5v" (path "/ec98644d-848c-5056-a4cb-c829189be5c3" (reference "H2") (unit 1))))
   )
-  (symbol (lib_id "Mechanical:MountingHole") (at 50.8 149.86 0.0) (unit 1)
-    (exclude_from_sim no) (in_bom no) (on_board yes) (dnp no)
-    (property "Reference" "H3" (at 49.53 146.05 0) (effects (font (size 1.27 1.27)) (justify right)))
-    (property "Value" "M3" (at 54.61 152.4 0) (effects (font (size 1.27 1.27)) (justify left) hide))
-    (property "Footprint" "MountingHole:MountingHole_3.2mm_M3" (at 50.8 149.86 0) (effects (font (size 1.27 1.27)) hide))
+  (symbol (lib_id "Mechanical:Fiducial") (at 50.8 149.86 0.0) (unit 1)
+    (exclude_from_sim no) (in_bom no) (on_board yes) (dnp no)
+    (property "Reference" "FID1" (at 49.53 146.05 0) (effects (font (size 1.27 1.27)) (justify right)))
+    (property "Value" "Fiducial" (at 54.61 152.4 0) (effects (font (size 1.27 1.27)) (justify left) hide))
+    (property "Footprint" "Fiducial:Fiducial_1mm_Mask2mm" (at 50.8 149.86 0) (effects (font (size 1.27 1.27)) hide))
     (property "Datasheet" "~" (at 50.8 149.86 0) (effects (font (size 1.27 1.27)) hide))
     (property "MPN" "n/a" (at 50.8 149.86 0) (effects (font (size 1.27 1.27)) hide))
     (property "Manufacturer" "n/a" (at 50.8 149.86 0) (effects (font (size 1.27 1.27)) hide))
-    (instances (project "buck-5v" (path "/ec98644d-848c-5056-a4cb-c829189be5c3" (reference "H3") (unit 1))))
+    (instances (project "buck-5v" (path "/ec98644d-848c-5056-a4cb-c829189be5c3" (reference "FID1") (unit 1))))
   )
   (symbol (lib_id "Mechanical:Fiducial") (at 63.5 149.86 0.0) (unit 1)
     (exclude_from_sim no) (in_bom no) (on_board yes) (dnp no)
-    (property "Reference" "FID1" (at 62.23 146.05 0) (effects (font (size 1.27 1.27)) (justify right)))
+    (property "Reference" "FID2" (at 62.23 146.05 0) (effects (font (size 1.27 1.27)) (justify right)))
     (property "Value" "Fiducial" (at 67.31 152.4 0) (effects (font (size 1.27 1.27)) (justify left) hide))
     (property "Footprint" "Fiducial:Fiducial_1mm_Mask2mm" (at 63.5 149.86 0) (effects (font (size 1.27 1.27)) hide))
@@
     (property "MPN" "n/a" (at 63.5 149.86 0) (effects (font (size 1.27 1.27)) hide))
     (property "Manufacturer" "n/a" (at 63.5 149.86 0) (effects (font (size 1.27 1.27)) hide))
-    (instances (project "buck-5v" (path "/ec98644d-848c-5056-a4cb-c829189be5c3" (reference "FID1") (unit 1))))
-  )
-  (symbol (lib_id "Mechanical:Fiducial") (at 76.2 149.86 0.0) (unit 1)
-    (exclude_from_sim no) (in_bom no) (on_board yes) (dnp no)
-    (property "Reference" "FID2" (at 74.93 146.05 0) (effects (font (size 1.27 1.27)) (justify right)))
+    (instances (project "buck-5v" (path "/ec98644d-848c-5056-a4cb-c829189be5c3" (reference "FID2") (unit 1))))
+  )
+  (symbol (lib_id "Mechanical:Fiducial") (at 76.19999999999999 149.86 0.0) (unit 1)
+    (exclude_from_sim no) (in_bom no) (on_board yes) (dnp no)
+    (property "Reference" "FID3" (at 74.93 146.05 0) (effects (font (size 1.27 1.27)) (justify right)))
     (property "Value" "Fiducial" (at 80.01 152.4 0) (effects (font (size 1.27 1.27)) (justify left) hide))
-    (property "Footprint" "Fiducial:Fiducial_1mm_Mask2mm" (at 76.2 149.86 0) (effects (font (size 1.27 1.27)) hide))
-    (property "Datasheet" "~" (at 76.2 149.86 0) (effects (font (size 1.27 1.27)) hide))
-    (property "MPN" "n/a" (at 76.2 149.86 0) (effects (font (size 1.27 1.27)) hide))
-    (property "Manufacturer" "n/a" (at 76.2 149.86 0) (effects (font (size 1.27 1.27)) hide))
-    (instances (project "buck-5v" (path "/ec98644d-848c-5056-a4cb-c829189be5c3" (reference "FID2") (unit 1))))
-  )
-  (symbol (lib_id "Mechanical:Fiducial") (at 88.9 149.86 0.0) (unit 1)
-    (exclude_from_sim no) (in_bom no) (on_board yes) (dnp no)
-    (property "Reference" "FID3" (at 87.63 146.05 0) (effects (font (size 1.27 1.27)) (justify right)))
-    (property "Value" "Fiducial" (at 92.71 152.4 0) (effects (font (size 1.27 1.27)) (justify left) hide))
-    (property "Footprint" "Fiducial:Fiducial_1mm_Mask2mm" (at 88.9 149.86 0) (effects (font (size 1.27 1.27)) hide))
-    (property "Datasheet" "~" (at 88.9 149.86 0) (effects (font (size 1.27 1.27)) hide))
-    (property "MPN" "n/a" (at 88.9 149.86 0) (effects (font (size 1.27 1.27)) hide))
-    (property "Manufacturer" "n/a" (at 88.9 149.86 0) (effects (font (size 1.27 1.27)) hide))
+    (property "Footprint" "Fiducial:Fiducial_1mm_Mask2mm" (at 76.19999999999999 149.86 0) (effects (font (size 1.27 1.27)) hide))
+    (property "Datasheet" "~" (at 76.19999999999999 149.86 0) (effects (font (size 1.27 1.27)) hide))
+    (property "MPN" "n/a" (at 76.19999999999999 149.86 0) (effects (font (size 1.27 1.27)) hide))
+    (property "Manufacturer" "n/a" (at 76.19999999999999 149.86 0) (effects (font (size 1.27 1.27)) hide))
     (instances (project "buck-5v" (path "/ec98644d-848c-5056-a4cb-c829189be5c3" (reference "FID3") (unit 1))))
   )
