File: examples/buck-5v/reviewed/buck-5v.kicad_sch (KiCad schematic)
At the start: 18 parts, among them J1 12V IN, J2 5V OUT, U1 LM2596S-5

Commit message: Put the vias back where the copper moved, and let the fillets vote
The FPGA board came back from its re-route with two unconnected nets and
three dangling ends, and the cause was older than anything this round
added. The router hands back a via for every layer change; six passes
then reshape the copper - snapping to 45s, chamfering, spreading folds,
and now filleting - and none of them move the holes underneath. A joint
that slides a millimetre from its via is two loose ends and one broken
net, and `_unlooped` then swept the via away as orphaned, because it
kept a via only when a track ended on its exact coordinate.

Two fixes, both about what "connected" means. A via lives if kept copper
*touches* it, not if a coordinate matches. And a new `_joined` pass
re-derives the joints from the copper that actually got written: where a
net ends on two layers at one point with no via reaching it, one goes
back in. It reads the finished geometry, so it cannot drift the way six
separate passes carrying vias along with them would.

The same reasoning fixes two rules that had been measuring coordinates
rather than copper. `route.stub` matched a track end to a via's centre
exactly, and called a joint a stub whenever a reshaping pass had moved
it a quarter of a millimetre inside the very barrel it was connected to.
`route.width_step` walked a neck back to its pad and stopped at the
first width change - which, on a filleted board, is the teardrop, so
every escape's neck stopped being recognised as one.

While the three copies of the post-route pipeline were being edited for
the third time this session, they became one function. That is how
`_teardrops` had come to run on two of the three exits.

All five boards: DRC clean on both matrix versions, nothing unconnected.
Four pass their gates; the FPGA board is down to the two-layer bill it
has always had - four nets over plane cuts and one 88 degree corner.

Co-Authored-By: Claude Fable 5 <noreply@anthropic.com>
Claude-Session: https:/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
Changed lines of the file:
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@@
     (exclude_from_sim no) (in_bom no) (on_board yes) (dnp no)
     (property "Reference" "H1" (at 24.13 146.05 0) (effects (font (size 1.27 1.27)) (justify right)))
-    (property "Value" "M3" (at 29.21 152.4 0) (effects (font (size 1.27 1.27)) (justify left)))
+    (property "Value" "M3" (at 29.21 152.4 0) (effects (font (size 1.27 1.27)) (justify left) hide))
     (property "Footprint" "MountingHole:MountingHole_3.2mm_M3" (at 25.4 149.86 0) (effects (font (size 1.27 1.27)) hide))
     (property "Datasheet" "~" (at 25.4 149.86 0) (effects (font (size 1.27 1.27)) hide))
@@
     (exclude_from_sim no) (in_bom no) (on_board yes) (dnp no)
     (property "Reference" "H2" (at 36.83 146.05 0) (effects (font (size 1.27 1.27)) (justify right)))
-    (property "Value" "M3" (at 41.91 152.4 0) (effects (font (size 1.27 1.27)) (justify left)))
+    (property "Value" "M3" (at 41.91 152.4 0) (effects (font (size 1.27 1.27)) (justify left) hide))
     (property "Footprint" "MountingHole:MountingHole_3.2mm_M3" (at 38.099999999999994 149.86 0) (effects (font (size 1.27 1.27)) hide))
     (property "Datasheet" "~" (at 38.099999999999994 149.86 0) (effects (font (size 1.27 1.27)) hide))
@@
     (exclude_from_sim no) (in_bom no) (on_board yes) (dnp no)
     (property "Reference" "H3" (at 49.53 146.05 0) (effects (font (size 1.27 1.27)) (justify right)))
-    (property "Value" "M3" (at 54.61 152.4 0) (effects (font (size 1.27 1.27)) (justify left)))
+    (property "Value" "M3" (at 54.61 152.4 0) (effects (font (size 1.27 1.27)) (justify left) hide))
     (property "Footprint" "MountingHole:MountingHole_3.2mm_M3" (at 50.8 149.86 0) (effects (font (size 1.27 1.27)) hide))
     (property "Datasheet" "~" (at 50.8 149.86 0) (effects (font (size 1.27 1.27)) hide))
@@
     (exclude_from_sim no) (in_bom no) (on_board yes) (dnp no)
     (property "Reference" "H4" (at 62.23 146.05 0) (effects (font (size 1.27 1.27)) (justify right)))
-    (property "Value" "M3" (at 67.31 152.4 0) (effects (font (size 1.27 1.27)) (justify left)))
+    (property "Value" "M3" (at 67.31 152.4 0) (effects (font (size 1.27 1.27)) (justify left) hide))
     (property "Footprint" "MountingHole:MountingHole_3.2mm_M3" (at 63.49999999999999 149.86 0) (effects (font (size 1.27 1.27)) hide))
     (property "Datasheet" "~" (at 63.49999999999999 149.86 0) (effects (font (size 1.27 1.27)) hide))
@@
     (exclude_from_sim no) (in_bom no) (on_board yes) (dnp no)
     (property "Reference" "FID1" (at 74.93 146.05 0) (effects (font (size 1.27 1.27)) (justify right)))
-    (property "Value" "Fiducial" (at 80.01 152.4 0) (effects (font (size 1.27 1.27)) (justify left)))
+    (property "Value" "Fiducial" (at 80.01 152.4 0) (effects (font (size 1.27 1.27)) (justify left) hide))
     (property "Footprint" "Fiducial:Fiducial_1mm_Mask2mm" (at 76.2 149.86 0) (effects (font (size 1.27 1.27)) hide))
     (property "Datasheet" "~" (at 76.2 149.86 0) (effects (font (size 1.27 1.27)) hide))
@@
     (exclude_from_sim no) (in_bom no) (on_board yes) (dnp no)
     (property "Reference" "FID2" (at 87.63 146.05 0) (effects (font (size 1.27 1.27)) (justify right)))
-    (property "Value" "Fiducial" (at 92.71 152.4 0) (effects (font (size 1.27 1.27)) (justify left)))
+    (property "Value" "Fiducial" (at 92.71 152.4 0) (effects (font (size 1.27 1.27)) (justify left) hide))
     (property "Footprint" "Fiducial:Fiducial_1mm_Mask2mm" (at 88.9 149.86 0) (effects (font (size 1.27 1.27)) hide))
     (property "Datasheet" "~" (at 88.9 149.86 0) (effects (font (size 1.27 1.27)) hide))
@@
     (exclude_from_sim no) (in_bom no) (on_board yes) (dnp no)
     (property "Reference" "FID3" (at 100.33 146.05 0) (effects (font (size 1.27 1.27)) (justify right)))
-    (property "Value" "Fiducial" (at 105.41 152.4 0) (effects (font (size 1.27 1.27)) (justify left)))
+    (property "Value" "Fiducial" (at 105.41 152.4 0) (effects (font (size 1.27 1.27)) (justify left) hide))
     (property "Footprint" "Fiducial:Fiducial_1mm_Mask2mm" (at 101.6 149.86 0) (effects (font (size 1.27 1.27)) hide))
     (property "Datasheet" "~" (at 101.6 149.86 0) (effects (font (size 1.27 1.27)) hide))

Commit message: Leave room for the screw, and print the ink where the board is
The screw holes were placed against the hole's own courtyard, which is the
drill plus a whisker - so on four of the five boards a hole sat inside a
connector's mating space, closest 0.42 mm. What goes through an M3 hole is a
pan head on a washer, seven millimetres of steel lying flat, and a connector
wants its shell, its wires and the fingers that fit them on top of that. The
spot search now keeps the fastener's own circle clear of every part body and
gives connectors CONNECTOR_ACCESS more, and three rules say so when a board
does not: mechanical.fastener_clearance, mechanical.connector_access and
mechanical.fastener_copper, all blocking for a generated design.

Silk was measured with a per-character advance of 0.78, and KiCad's stroke
font is proportional at 0.94 to 1.07. Everything downstream of that estimate
was placing ink where it did not fit: a legend across a capacitor's land, a
designator through the board's own name. `_text_extent` takes the top of the
measured range, adds the fab's clearance and is used by every silk placement.

Three placements also fell through to a position nobody chose. A designator
that found nothing kept its library offset, which for a part in a corner
points off the board; the board id took the first of eight fixed strips; a
legend took the least bad of six spots. All three are scored now, over
candidate sets wide enough to have an answer - and a pad-less footprint, which
is what a mounting hole is, is no longer skipped outright.

silk.off_board reports the case KiCad's own test cannot: ink that clears the
edge entirely is never printed, and DRC only measures ink that crosses it.

_unspiked redraws a corner tighter than a right angle as the elbow between its
neighbours - one diagonal, one straight, no step back to a heading the line
has already left. It is never longer than what it replaces.

All four fast boards: 0 errors, 0 warnings.

Co-Authored-By: Claude Fable 5 <no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
Parts:
- removed H3, H4: M3, MountingHole:MountingHole_3.2mm_M3, symbol Mechanical:MountingHole
Other:
- moved on the sheet: FID1, FID2, FID3
Changed lines of the file:
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@@
     (instances (project "buck-5v" (path "/ec98644d-848c-5056-a4cb-c829189be5c3" (reference "H2") (unit 1))))
   )
-  (symbol (lib_id "Mechanical:MountingHole") (at 50.8 149.86 0.0) (unit 1)
+  (symbol (lib_id "Mechanical:Fiducial") (at 50.8 149.86 0.0) (unit 1)
     (exclude_from_sim no) (in_bom no) (on_board yes) (dnp no)
-    (property "Reference" "H3" (at 49.53 146.05 0) (effects (font (size 1.27 1.27)) (justify right)))
-    (property "Value" "M3" (at 54.61 152.4 0) (effects (font (size 1.27 1.27)) (justify left) hide))
-    (property "Footprint" "MountingHole:MountingHole_3.2mm_M3" (at 50.8 149.86 0) (effects (font (size 1.27 1.27)) hide))
+    (property "Reference" "FID1" (at 49.53 146.05 0) (effects (font (size 1.27 1.27)) (justify right)))
+    (property "Value" "Fiducial" (at 54.61 152.4 0) (effects (font (size 1.27 1.27)) (justify left) hide))
+    (property "Footprint" "Fiducial:Fiducial_1mm_Mask2mm" (at 50.8 149.86 0) (effects (font (size 1.27 1.27)) hide))
     (property "Datasheet" "~" (at 50.8 149.86 0) (effects (font (size 1.27 1.27)) hide))
     (property "MPN" "n/a" (at 50.8 149.86 0) (effects (font (size 1.27 1.27)) hide))
     (property "Manufacturer" "n/a" (at 50.8 149.86 0) (effects (font (size 1.27 1.27)) hide))
-    (instances (project "buck-5v" (path "/ec98644d-848c-5056-a4cb-c829189be5c3" (reference "H3") (unit 1))))
-  )
-  (symbol (lib_id "Mechanical:MountingHole") (at 63.49999999999999 149.86 0.0) (unit 1)
-    (exclude_from_sim no) (in_bom no) (on_board yes) (dnp no)
-    (property "Reference" "H4" (at 62.23 146.05 0) (effects (font (size 1.27 1.27)) (justify right)))
-    (property "Value" "M3" (at 67.31 152.4 0) (effects (font (size 1.27 1.27)) (justify left) hide))
-    (property "Footprint" "MountingHole:MountingHole_3.2mm_M3" (at 63.49999999999999 149.86 0) (effects (font (size 1.27 1.27)) hide))
-    (property "Datasheet" "~" (at 63.49999999999999 149.86 0) (effects (font (size 1.27 1.27)) hide))
-    (property "MPN" "n/a" (at 63.49999999999999 149.86 0) (effects (font (size 1.27 1.27)) hide))
-    (property "Manufacturer" "n/a" (at 63.49999999999999 149.86 0) (effects (font (size 1.27 1.27)) hide))
-    (instances (project "buck-5v" (path "/ec98644d-848c-5056-a4cb-c829189be5c3" (reference "H4") (unit 1))))
-  )
-  (symbol (lib_id "Mechanical:Fiducial") (at 76.2 149.86 0.0) (unit 1)
-    (exclude_from_sim no) (in_bom no) (on_board yes) (dnp no)
-    (property "Reference" "FID1" (at 74.93 146.05 0) (effects (font (size 1.27 1.27)) (justify right)))
-    (property "Value" "Fiducial" (at 80.01 152.4 0) (effects (font (size 1.27 1.27)) (justify left) hide))
-    (property "Footprint" "Fiducial:Fiducial_1mm_Mask2mm" (at 76.2 149.86 0) (effects (font (size 1.27 1.27)) hide))
-    (property "Datasheet" "~" (at 76.2 149.86 0) (effects (font (size 1.27 1.27)) hide))
-    (property "MPN" "n/a" (at 76.2 149.86 0) (effects (font (size 1.27 1.27)) hide))
-    (property "Manufacturer" "n/a" (at 76.2 149.86 0) (effects (font (size 1.27 1.27)) hide))
     (instances (project "buck-5v" (path "/ec98644d-848c-5056-a4cb-c829189be5c3" (reference "FID1") (unit 1))))
   )
-  (symbol (lib_id "Mechanical:Fiducial") (at 88.9 149.86 0.0) (unit 1)
+  (symbol (lib_id "Mechanical:Fiducial") (at 63.5 149.86 0.0) (unit 1)
     (exclude_from_sim no) (in_bom no) (on_board yes) (dnp no)
-    (property "Reference" "FID2" (at 87.63 146.05 0) (effects (font (size 1.27 1.27)) (justify right)))
-    (property "Value" "Fiducial" (at 92.71 152.4 0) (effects (font (size 1.27 1.27)) (justify left) hide))
-    (property "Footprint" "Fiducial:Fiducial_1mm_Mask2mm" (at 88.9 149.86 0) (effects (font (size 1.27 1.27)) hide))
-    (property "Datasheet" "~" (at 88.9 149.86 0) (effects (font (size 1.27 1.27)) hide))
-    (property "MPN" "n/a" (at 88.9 149.86 0) (effects (font (size 1.27 1.27)) hide))
-    (property "Manufacturer" "n/a" (at 88.9 149.86 0) (effects (font (size 1.27 1.27)) hide))
+    (property "Reference" "FID2" (at 62.23 146.05 0) (effects (font (size 1.27 1.27)) (justify right)))
+    (property "Value" "Fiducial" (at 67.31 152.4 0) (effects (font (size 1.27 1.27)) (justify left) hide))
+    (property "Footprint" "Fiducial:Fiducial_1mm_Mask2mm" (at 63.5 149.86 0) (effects (font (size 1.27 1.27)) hide))
+    (property "Datasheet" "~" (at 63.5 149.86 0) (effects (font (size 1.27 1.27)) hide))
+    (property "MPN" "n/a" (at 63.5 149.86 0) (effects (font (size 1.27 1.27)) hide))
+    (property "Manufacturer" "n/a" (at 63.5 149.86 0) (effects (font (size 1.27 1.27)) hide))
     (instances (project "buck-5v" (path "/ec98644d-848c-5056-a4cb-c829189be5c3" (reference "FID2") (unit 1))))
   )
-  (symbol (lib_id "Mechanical:Fiducial") (at 101.6 149.86 0.0) (unit 1)
+  (symbol (lib_id "Mechanical:Fiducial") (at 76.19999999999999 149.86 0.0) (unit 1)
     (exclude_from_sim no) (in_bom no) (on_board yes) (dnp no)
-    (property "Reference" "FID3" (at 100.33 146.05 0) (effects (font (size 1.27 1.27)) (justify right)))
-    (property "Value" "Fiducial" (at 105.41 152.4 0) (effects (font (size 1.27 1.27)) (justify left) hide))
-    (property "Footprint" "Fiducial:Fiducial_1mm_Mask2mm" (at 101.6 149.86 0) (effects (font (size 1.27 1.27)) hide))
-    (property "Datasheet" "~" (at 101.6 149.86 0) (effects (font (size 1.27 1.27)) hide))
-    (property "MPN" "n/a" (at 101.6 149.86 0) (effects (font (size 1.27 1.27)) hide))
-    (property "Manufacturer" "n/a" (at 101.6 149.86 0) (effects (font (size 1.27 1.27)) hide))
+    (property "Reference" "FID3" (at 74.93 146.05 0) (effects (font (size 1.27 1.27)) (justify right)))
+    (property "Value" "Fiducial" (at 80.01 152.4 0) (effects (font (size 1.27 1.27)) (justify left) hide))
+    (property "Footprint" "Fiducial:Fiducial_1mm_Mask2mm" (at 76.19999999999999 149.86 0) (effects (font (size 1.27 1.27)) hide))
+    (property "Datasheet" "~" (at 76.19999999999999 149.86 0) (effects (font (size 1.27 1.27)) hide))
+    (property "MPN" "n/a" (at 76.19999999999999 149.86 0) (effects (font (size 1.27 1.27)) hide))
+    (property "Manufacturer" "n/a" (at 76.19999999999999 149.86 0) (effects (font (size 1.27 1.27)) hide))
     (instances (project "buck-5v" (path "/ec98644d-848c-5056-a4cb-c829189be5c3" (reference "FID3") (unit 1))))
   )

Commit message: Walk the whole edge for a screw hole, and land a joint on its own pad
The fastener clearance was right and the search was not: it slid along two
edges from each corner and gave up, so boards that had had four screw holes
came back with one. It now walks a ring round the board at the inset the
screw needs, taking the nearest free point to each corner - and only from
that corner's own quarter, because a search that asked for the nearest free
point anywhere put three of the four along one edge, each of them the nearest
thing to a different corner. A quarter with no room gives no screw: three
that hold the board flat beat four that hold one side.

A pin header asks for nothing above its courtyard - the socket that fits it
lands inside the outline the header already draws - while a screw terminal's
wires leave horizontally from its face. Treating the two alike is what left a
carrier lined with headers with two holes on one edge. Both the generator and
the rule now tell them apart by footprint.

_landed folds a via that sits beside a plated hole of its own net onto the
hole. The plating already joins the faces, so the via bought nothing and cost
hole-to-hole: two drills a millimetre apart leave 0.15 mm of laminate at a
0.25 mm rule, which is what DRC reported on the opamp board.

The fillets move to the end of the pipeline. A taper is built against the end
of a run, and _landed moves ends, so a teardrop laid before it pointed at
where the run used to stop - a nought-degree corner in the angle rule.

buck-5v, motor-driver, pico-carrier, opamp-filter: 0 errors, 0 warnings.

Co-Authored-By: Claude Fable 5 <noreply@anthropic.com>
Claude-Session: https://claude.ai/code/session_01DUj7Ltu92tWg159mCSacwY
Parts:
- added H3: M3, MountingHole:MountingHole_3.2mm_M3, symbol Mechanical:MountingHole
Other:
- moved on the sheet: FID1, FID2, FID3
Changed lines of the file:
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@@
     (instances (project "buck-5v" (path "/ec98644d-848c-5056-a4cb-c829189be5c3" (reference "H2") (unit 1))))
   )
-  (symbol (lib_id "Mechanical:Fiducial") (at 50.8 149.86 0.0) (unit 1)
+  (symbol (lib_id "Mechanical:MountingHole") (at 50.8 149.86 0.0) (unit 1)
     (exclude_from_sim no) (in_bom no) (on_board yes) (dnp no)
-    (property "Reference" "FID1" (at 49.53 146.05 0) (effects (font (size 1.27 1.27)) (justify right)))
-    (property "Value" "Fiducial" (at 54.61 152.4 0) (effects (font (size 1.27 1.27)) (justify left) hide))
-    (property "Footprint" "Fiducial:Fiducial_1mm_Mask2mm" (at 50.8 149.86 0) (effects (font (size 1.27 1.27)) hide))
+    (property "Reference" "H3" (at 49.53 146.05 0) (effects (font (size 1.27 1.27)) (justify right)))
+    (property "Value" "M3" (at 54.61 152.4 0) (effects (font (size 1.27 1.27)) (justify left) hide))
+    (property "Footprint" "MountingHole:MountingHole_3.2mm_M3" (at 50.8 149.86 0) (effects (font (size 1.27 1.27)) hide))
     (property "Datasheet" "~" (at 50.8 149.86 0) (effects (font (size 1.27 1.27)) hide))
     (property "MPN" "n/a" (at 50.8 149.86 0) (effects (font (size 1.27 1.27)) hide))
     (property "Manufacturer" "n/a" (at 50.8 149.86 0) (effects (font (size 1.27 1.27)) hide))
-    (instances (project "buck-5v" (path "/ec98644d-848c-5056-a4cb-c829189be5c3" (reference "FID1") (unit 1))))
+    (instances (project "buck-5v" (path "/ec98644d-848c-5056-a4cb-c829189be5c3" (reference "H3") (unit 1))))
   )
   (symbol (lib_id "Mechanical:Fiducial") (at 63.5 149.86 0.0) (unit 1)
     (exclude_from_sim no) (in_bom no) (on_board yes) (dnp no)
-    (property "Reference" "FID2" (at 62.23 146.05 0) (effects (font (size 1.27 1.27)) (justify right)))
+    (property "Reference" "FID1" (at 62.23 146.05 0) (effects (font (size 1.27 1.27)) (justify right)))
     (property "Value" "Fiducial" (at 67.31 152.4 0) (effects (font (size 1.27 1.27)) (justify left) hide))
     (property "Footprint" "Fiducial:Fiducial_1mm_Mask2mm" (at 63.5 149.86 0) (effects (font (size 1.27 1.27)) hide))
@@
     (property "MPN" "n/a" (at 63.5 149.86 0) (effects (font (size 1.27 1.27)) hide))
     (property "Manufacturer" "n/a" (at 63.5 149.86 0) (effects (font (size 1.27 1.27)) hide))
+    (instances (project "buck-5v" (path "/ec98644d-848c-5056-a4cb-c829189be5c3" (reference "FID1") (unit 1))))
+  )
+  (symbol (lib_id "Mechanical:Fiducial") (at 76.2 149.86 0.0) (unit 1)
+    (exclude_from_sim no) (in_bom no) (on_board yes) (dnp no)
+    (property "Reference" "FID2" (at 74.93 146.05 0) (effects (font (size 1.27 1.27)) (justify right)))
+    (property "Value" "Fiducial" (at 80.01 152.4 0) (effects (font (size 1.27 1.27)) (justify left) hide))
+    (property "Footprint" "Fiducial:Fiducial_1mm_Mask2mm" (at 76.2 149.86 0) (effects (font (size 1.27 1.27)) hide))
+    (property "Datasheet" "~" (at 76.2 149.86 0) (effects (font (size 1.27 1.27)) hide))
+    (property "MPN" "n/a" (at 76.2 149.86 0) (effects (font (size 1.27 1.27)) hide))
+    (property "Manufacturer" "n/a" (at 76.2 149.86 0) (effects (font (size 1.27 1.27)) hide))
     (instances (project "buck-5v" (path "/ec98644d-848c-5056-a4cb-c829189be5c3" (reference "FID2") (unit 1))))
   )
-  (symbol (lib_id "Mechanical:Fiducial") (at 76.19999999999999 149.86 0.0) (unit 1)
+  (symbol (lib_id "Mechanical:Fiducial") (at 88.9 149.86 0.0) (unit 1)
     (exclude_from_sim no) (in_bom no) (on_board yes) (dnp no)
-    (property "Reference" "FID3" (at 74.93 146.05 0) (effects (font (size 1.27 1.27)) (justify right)))
-    (property "Value" "Fiducial" (at 80.01 152.4 0) (effects (font (size 1.27 1.27)) (justify left) hide))
-    (property "Footprint" "Fiducial:Fiducial_1mm_Mask2mm" (at 76.19999999999999 149.86 0) (effects (font (size 1.27 1.27)) hide))
-    (property "Datasheet" "~" (at 76.19999999999999 149.86 0) (effects (font (size 1.27 1.27)) hide))
-    (property "MPN" "n/a" (at 76.19999999999999 149.86 0) (effects (font (size 1.27 1.27)) hide))
-    (property "Manufacturer" "n/a" (at 76.19999999999999 149.86 0) (effects (font (size 1.27 1.27)) hide))
+    (property "Reference" "FID3" (at 87.63 146.05 0) (effects (font (size 1.27 1.27)) (justify right)))
+    (property "Value" "Fiducial" (at 92.71 152.4 0) (effects (font (size 1.27 1.27)) (justify left) hide))
+    (property "Footprint" "Fiducial:Fiducial_1mm_Mask2mm" (at 88.9 149.86 0) (effects (font (size 1.27 1.27)) hide))
+    (property "Datasheet" "~" (at 88.9 149.86 0) (effects (font (size 1.27 1.27)) hide))
+    (property "MPN" "n/a" (at 88.9 149.86 0) (effects (font (size 1.27 1.27)) hide))
+    (property "Manufacturer" "n/a" (at 88.9 149.86 0) (effects (font (size 1.27 1.27)) hide))
     (instances (project "buck-5v" (path "/ec98644d-848c-5056-a4cb-c829189be5c3" (reference "FID3") (unit 1))))
   )
