File: examples/buck-5v/reviewed/buck-5v.kicad_sch (KiCad schematic)
At the start: 16 parts, among them J1 12V IN, J2 5V OUT, U1 LM2596S-5

Commit message: chore(examples): regenerate the four two-layer boards and their pictures
buck-5v, motor-driver, pico-carrier and opamp-filter, regenerated from the
merged generator and gated clean on KiCad 9.0.9. The inner-layer pictures go
with the inner layers.

fpga-audio is still routing; it follows.

Co-Authored-By: Claude Opus 5 <noreply@anthropic.com>
Claude-Session: https://claude.ai/code/session_01XQE7UkE9WTSMW3oZ3kLeCt
Parts:
- added D3: SMAJ18A, Diode_SMD:D_SMA, symbol Device:D_Zener
- added F1: 3A, Fuse:Fuse_1206_3216Metric, symbol Device:Fuse
- C3: ESR (none) -> 150mR max @100kHz
Connections:
- net +12V: now also D3.1 (K), F1.2; no longer J1.1 (Pin_1)
- net GND: now also D3.2 (A)
- new net VIN: F1.1, J1.1 (Pin_1)
Other:
- note added: "C1 220u/35V bulk, C2 100n/50V bypass - both above 1.5x the 12 V."
- note added: "C3's ESR is part of the design: 0.6 A x 150 mR = 90 mV"
- note added: "Input: F1 3 A opens on a fault or reversed leads; D3 clamps"
- note added: "above 18 V and is the diode the reversed supply flows through."
- note added: "capacitor - an all-ceramic substitute rings."
- note added: "ripple, and the LM2596 loop needs ESR in the output"
- note removed: "Input: C1 220u/35V bulk, C2 100n/50V bypass -"
- note removed: "both above 1.5x the 12 V they sit on."
- moved on the sheet: C1, J1
