File: examples/pico-carrier/as-generated/pico-carrier.kicad_sch (KiCad schematic)
At the start: 14 parts, among them J1 5V IN, J3 GP0-GP15, J4 GP16-GP28, PWR, U1 Pico

Commit message: chore(examples): regenerate the four two-layer boards and their pictures
buck-5v, motor-driver, pico-carrier and opamp-filter, regenerated from the
merged generator and gated clean on KiCad 9.0.9. The inner-layer pictures go
with the inner layers.

fpga-audio is still routing; it follows.

Co-Authored-By: Claude Opus 5 <noreply@anthropic.com>
Claude-Session: https://claude.ai/code/session_01XQE7UkE9WTSMW3oZ3kLeCt
Parts:
- added F1: 0.75A, Fuse:Fuse_1812_4532Metric, symbol Device:Polyfuse
Connections:
- net +5V: now also F1.2; no longer D1.2 (A)
- new net 5V_FUSED: D1.2 (A), F1.1
Other:
- moved on the sheet: D1, J1
